File: ISOpowerPCB/B_usb_interface.kicad_sch (KiCad schematic)
At the start: 19 parts

Commit message: modified pcb files
Parts:
- removed C? (x3): 100n, Capacitor_SMD:C_0805_2012Metric_Pad1.18x1.45mm_HandSolder, symbol 000_Capacitor_film_immo:cap_film_0805
- removed C?: 4n7, Capacitor_SMD:C_0805_2012Metric_Pad1.18x1.45mm_HandSolder, symbol 000_Capacitor_film_immo:cap_film_0805
- removed D?: PRTR5V0U2X, Package_TO_SOT_SMD:SOT-143, symbol Power_Protection:PRTR5V0U2X
- removed J?: USB_B_Mini, symbol Connector:USB_B_Mini
- removed R?: 1M, Resistor_SMD:R_0805_2012Metric_Pad1.20x1.40mm_HandSolder, symbol 000_Resistors_Immo:Resistor_0805
- removed TP? (x2): TestPoint, symbol Connector:TestPoint
- removed U?: CH340C, Package_SO:SOIC-16_3.9x9.9mm_P1.27mm, symbol Interface_USB:CH340C
Connections:
- no-connect marks 2 -> 1
Other:
- note added: "3.3v USB Interface"
- note removed: "5v USB Interface"
- note removed: "USB power routed to its own bus, to allow potential for USB power to be used for powering microcontrollers during programming, but avoid case where user inadvertently tries to power entire 5v BUS from USB rail"
- moved on the sheet: C?, D?, J?, R?, TP?, U?
