File: ISOpowerPCB/v_monitor.kicad_sch (KiCad schematic)
At the start: 20 parts

Commit message: Updated as per discussions 26/01/22
# Change Notes

04/02/2022
As per discussion 26/01/22
1. Changed per channel 5v MOSFET switches to MOSFET control of DC/DC module on/off pin - due to failure of MOSFET switching during testing.
2. Added 5v buck converter for independent MCU_5V power bus.
	- Ensured all 5v MCU hardware is powered from common MCU_5V bus.
3. Removed circuit from NC pins on DC/DC modules.
4. Changed ESP32 USB interface to CH340
5. Changed MCU serial logic level converters from MOSFET to IC - TXS0102DCT
	- TODO: OE pin now requires low signal untill DC/DC supply is stable - Does it? Can it just be tied to 5v bus with a large capacitor? Does it need MCU to hold pin low untill 5V_BUS is stable?
6. Removed redundent 3V3_IN to power distribution page.
	- Rechecked all sheets for redundent pins, it won't impact drawing traces, but it will impact readability.
7. Added Mechanical layer as hirarchical sheet.
8. Moved voltage monitoring circuits to hirarchical sheet
9. Added voltage monitoring with TL431DBZ to 12V_BUS
10. Automatic shutoff circuit removed, as this would prevent the DC/DC module from powering on. Instead moved to AtMega328p digital inputs
and microcontroller will control shutdown of DC/DC supply if out of spec voltage detected.
		- This is a severe limitation compared to the specification, and this also does not prevent damage to devices on 5V_BUS if voltage is pulled high, for example to 12v due to user error.
		- TODO: Add independent overvoltage protection to 5V_BUS? 		[Zener Diode Overvoltage Protection - Sparkfun](https://www.rs-online.com/designspark/how-does-zener-diode-do-overvoltage-protection-in-circuit#:~:text=In%20order%20to%20protect%20the,flow%20in%20the%20reverse%20direction).
11. Changed logic level conversion for 12v outputs to 12v drive circuit. [12v drive circuit](https://forum.arduino.cc/t/easiest-way-of-driving-amplifying-from-5v-to-12v/123290)
12. Added proto pin connections for ESP MCU.
13. Changed 20v Zener in reverse vol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
Changed lines of the file:
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@@
     (effects (font (size 0.8 0.8)) (justify left bottom))
   )
-  (hierarchical_label "GND_IN" (shape bidirectional) (at 25.4 21.59 180)
+  (hierarchical_label "GND_IN" (shape passive) (at 25.4 21.59 180)
     (effects (font (size 1.27 1.27)) (justify right))
   )

Commit message: messing around with libraries
Parts:
- gave numbers to parts that had none: 12
- renumbered R1a to R1a1, R1b to R1b1, R2a to R2a1, R2b to R2b1, R3a to R3a1, R3b to R3b1, R4a to R4a1, R4b to R4b1
Changed lines of the file:
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@@
     (effects (font (size 3 3)) (justify left bottom))
-  )
-  (text "Is it worth including this circuit for 12v sense as well? future use?"
-    (at 57.15 44.45 0)
-    (effects (font (size 0.8 0.8)) (justify left bottom))
   )
   (text "Outputs Logic HIGH when\n4.5v > Vbus > 5.5v " (at 59.69 40.64 0)
@@
   (symbol (lib_id "000_Connectors_Immo:Jumper_3_Bridged12") (at 133.35 36.83 0) (unit 1)
     (in_bom yes) (on_board yes) (fields_autoplaced)
-    (property "Reference" "JP?" (id 0) (at 133.35 31.75 0))
+    (property "Reference" "JP9" (id 0) (at 133.35 31.75 0))
     (property "Value" "5v Bus Monitor Disable" (id 1) (at 133.35 34.29 0))
     (property "Footprint" "" (id 2) (at 133.35 36.83 0)
@@
   (symbol (lib_id "000_Resistors_Immo:Resistor_0805") (at 149.86 111.76 90) (unit 1)
     (in_bom yes) (on_board yes) (fields_autoplaced)
-    (property "Reference" "R?" (id 0) (at 149.86 105.41 90))
+    (property "Reference" "R30" (id 0) (at 149.86 105.41 90))
     (property "Value" "10k" (id 1) (at 149.86 107.95 90))
     (property "Footprint" "Resistor_SMD:R_0805_2012Metric_Pad1.20x1.40mm_HandSolder" (id 2) (at 149.86 113.538 90)
@@
   (symbol (lib_id "000_Resistors_Immo:Resistor_0805") (at 99.06 54.61 0) (unit 1)
     (in_bom yes) (on_board yes) (fields_autoplaced)
-    (property "Reference" "R3b" (id 0) (at 101.6 53.3399 0)
+    (property "Reference" "R3b1" (id 0) (at 101.6 53.3399 0)
       (effects (font (size 1.27 1.27)) (justify left))
     )
@@
   (symbol (lib_id "Reference_Voltage:TL431DBZ") (at 109.22 135.89 90) (unit 1)
     (in_bom yes) (on_board yes)
-    (property "Reference" "U?" (id 0) (at 111.76 134.6199 90)
+    (property "Reference" "U18" (id 0) (at 111.76 134.6199 90)
       (effects (font (size 1.27 1.27)) (justify right))
     )
@@
   (symbol (lib_id "000_Resistors_Immo:Resistor_0805") (at 73.66 147.32 0) (unit 1)
     (in_bom yes) (on_board yes) (fields_autoplaced)
-    (property "Reference" "R2a" (id 0) (at 76.2 146.0499 0)
+    (property "Reference" "R2a1" (id 0) (at 76.2 146.0499 0)
       (effects (font (size 1.27 1.27)) (justify left))
     )
@@
   (symbol (lib_id "000_Resistors_Immo:Resistor_0805") (at 99.06 72.39 0) (unit 1)
     (in_bom yes) (on_board yes) (fields_autoplaced)
-    (property "Reference" "R4b" (id 0) (at 101.6 71.1199 0)
+    (property "Reference" "R4b1" (id 0) (at 101.6 71.1199 0)
       (effects (font (size 1.27 1.27)) (justify left))
     )
@@
   (symbol (lib_id "power:GND") (at 160.02 36.83 90) (unit 1)
     (in_bom yes) (on_board yes) (fields_autoplaced)
-    (property "Reference" "#PWR?" (id 0) (at 166.37 36.83 0)
+    (property "Reference" "#PWR091" (id 0) (at 166.37 36.83 0)
       (effects (font (size 1.27 1.27)) hide)
     )
@@
   (symbol (lib_id "Reference_Voltage:TL431DBZ") (at 85.09 140.97 90) (unit 1)
     (in_bom yes) (on_board yes) (fields_autoplaced)
-    (property "Reference" "U?" (id 0) (at 87.63 139.6999 90)
+    (property "Reference" "U16" (id 0) (at 87.63 139.6999 90)
       (effects (font (size 1.27 1.27)) (justify right))
     )
@@
   (symbol (lib_id "power:GND") (at 85.09 82.55 0) (unit 1)
     (in_bom yes) (on_board yes) (fields_autoplaced)
-    (property "Reference" "#PWR?" (id 0) (at 85.09 88.9 0)
+    (property "Reference" "#PWR089" (id 0) (at 85.09 88.9 0)
       (effects (font (size 1.27 1.27)) hide)
     )
@@
   (symbol (lib_id "Reference_Voltage:TL431DBZ") (at 109.22 60.96 90) (unit 1)
     (in_bom yes) (on_board yes)
-    (property "Reference" "U?" (id 0) (at 111.76 59.6899 90)
+    (property "Reference" "U17" (id 0) (at 111.76 59.6899 90)
       (effects (font (size 1.27 1.27)) (justify right))
     )
@@
   (symbol (lib_id "Connector:TestPoint") (at 125.73 36.83 180) (unit 1)
     (in_bom yes) (on_board yes)
-    (property "Reference" "TP?" (id 0) (at 121.92 40.64 0)
+    (property "Reference" "TP10" (id 0) (at 121.92 40.64 0)
       (effects (font (size 1.27 1.27)) (justify right))
     )
@@
   (symbol (lib_id "000_Resistors_Immo:Resistor_0805") (at 73.66 59.69 0) (unit 1)
     (in_bom yes) (on_board yes) (fields_autoplaced)
-    (property "Reference" "R1b" (id 0) (at 76.2 58.4199 0)
+    (property "Reference" "R1b1" (id 0) (at 76.2 58.4199 0)
       (effects (font (size 1.27 1.27)) (justify left))
     )
@@
   (symbol (lib_id "000_Resistors_Immo:Resistor_0805") (at 149.86 36.83 90) (unit 1)
     (in_bom yes) (on_board yes) (fields_autoplaced)
-    (property "Reference" "R?" (id 0) (at 149.86 30.48 90))
+    (property "Reference" "R29" (id 0) (at 149.86 30.48 90))
     (property "Value" "10k" (id 1) (at 149.86 33.02 90))
     (property "Footprint" "Resistor_SMD:R_0805_2012Metric_Pad1.20x1.40mm_HandSolder" (id 2) (at 149.86 38.608 90)
@@
   (symbol (lib_id "power:GND") (at 85.09 157.48 0) (unit 1)
     (in_bom yes) (on_board yes) (fields_autoplaced)
-    (property "Reference" "#PWR?" (id 0) (at 85.09 163.83 0)
+    (property "Reference" "#PWR090" (id 0) (at 85.09 163.83 0)
       (effects (font (size 1.27 1.27)) hide)
     )
@@
   (symbol (lib_id "Reference_Voltage:TL431DBZ") (at 85.09 66.04 90) (unit 1)
     (in_bom yes) (on_board yes) (fields_autoplaced)
-    (property "Reference" "U?" (id 0) (at 87.63 64.7699 90)
+    (property "Reference" "U15" (id 0) (at 87.63 64.7699 90)
       (effects (font (size 1.27 1.27)) (justify right))
     )
@@
   (symbol (lib_id "000_Resistors_Immo:Resistor_0805") (at 99.06 147.32 0) (unit 1)
     (in_bom yes) (on_board yes) (fields_autoplaced)
-    (property "Reference" "R4a" (id 0) (at 101.6 146.0499 0)
+    (property "Reference" "R4a1" (id 0) (at 101.6 146.0499 0)
       (effects (font (size 1.27 1.27)) (justify left))
     )
@@
   (symbol (lib_id "Connector:TestPoint") (at 116.84 109.22 0) (unit 1)
     (in_bom yes) (on_board yes)
-    (property "Reference" "TP?" (id 0) (at 120.65 105.41 0)
+    (property "Reference" "TP9" (id 0) (at 120.65 105.41 0)
       (effects (font (size 1.27 1.27)) (justify right))
     )
@@
   (symbol (lib_id "000_Resistors_Immo:Resistor_0805") (at 73.66 134.62 0) (unit 1)
     (in_bom yes) (on_board yes) (fields_autoplaced)
-    (property "Reference" "R1a" (id 0) (at 76.2 133.3499 0)
+    (property "Reference" "R1a1" (id 0) (at 76.2 133.3499 0)
       (effects (font (size 1.27 1.27)) (justify left))
     )
@@
   (symbol (lib_id "000_Connectors_Immo:Jumper_3_Bridged12") (at 133.35 111.76 0) (unit 1)
     (in_bom yes) (on_board yes) (fields_autoplaced)
-    (property "Reference" "JP?" (id 0) (at 133.35 106.68 0))
+    (property "Reference" "JP10" (id 0) (at 133.35 106.68 0))
     (property "Value" "12v Bus Monitor Disable" (id 1) (at 133.35 109.22 0))
     (property "Footprint" "" (id 2) (at 133.35 111.76 0)
@@
   (symbol (lib_id "000_Resistors_Immo:Resistor_0805") (at 99.06 129.54 0) (unit 1)
     (in_bom yes) (on_board yes) (fields_autoplaced)
-    (property "Reference" "R3a" (id 0) (at 101.6 128.2699 0)
+    (property "Reference" "R3a1" (id 0) (at 101.6 128.2699 0)
       (effects (font (size 1.27 1.27)) (justify left))
     )
@@
   (symbol (lib_id "power:GND") (at 160.02 111.76 90) (unit 1)
     (in_bom yes) (on_board yes) (fields_autoplaced)
-    (property "Reference" "#PWR?" (id 0) (at 166.37 111.76 0)
+    (property "Reference" "#PWR092" (id 0) (at 166.37 111.76 0)
       (effects (font (size 1.27 1.27)) hide)
     )
@@
   (symbol (lib_id "power:GND") (at 30.48 21.59 90) (unit 1)
     (in_bom yes) (on_board yes) (fields_autoplaced)
-    (property "Reference" "#PWR?" (id 0) (at 36.83 21.59 0)
+    (property "Reference" "#PWR088" (id 0) (at 36.83 21.59 0)
       (effects (font (size 1.27 1.27)) hide)
     )
@@
   (symbol (lib_id "000_Resistors_Immo:Resistor_0805") (at 109.22 46.99 0) (unit 1)
     (in_bom yes) (on_board yes) (fields_autoplaced)
-    (property "Reference" "R?" (id 0) (at 111.76 45.7199 0)
+    (property "Reference" "R27" (id 0) (at 111.76 45.7199 0)
       (effects (font (size 1.27 1.27)) (justify left))
     )
@@
   (symbol (lib_id "000_Resistors_Immo:Resistor_0805") (at 73.66 72.39 0) (unit 1)
     (in_bom yes) (on_board yes) (fields_autoplaced)
-    (property "Reference" "R2b" (id 0) (at 76.2 71.1199 0)
+    (property "Reference" "R2b1" (id 0) (at 76.2 71.1199 0)
       (effects (font (size 1.27 1.27)) (justify left))
     )
@@
   (symbol (lib_id "000_Resistors_Immo:Resistor_0805") (at 109.22 121.92 0) (unit 1)
     (in_bom yes) (on_board yes) (fields_autoplaced)
-    (property "Reference" "R?" (id 0) (at 111.76 120.6499 0)
-      (effects (font (size 1.27 1.27)) (justify left))
-    )
+    (property "Reference" "R28" (id 0) (at 111.76 120.6499 0)
+      (effects (font (size 1.27 1.27)) (justify left))
+    )
