File: ISOpowerPCB/v_monitor.kicad_sch (KiCad schematic)
At the start: 30 parts, among them U15 TL431DBZ, U16 TL431DBZ, U17 TL431DBZ, U18 TL431DBZ, U19 HEF4093B

Commit message: added documentation for component selection
Completed footprint association & added documentation re Netclasses. Need to update netclasses in schematic settings before moving to PCB layout.
Parts:
- JP10, JP9: footprint (none) -> Jumper:SolderJumper-3_P1.3mm_Bridged12_Pad1.0x1.5mm
- TP10, TP9: footprint (none) -> TestPoint:TestPoint_Pad_D1.5mm
- U19: footprint (none) -> Package_SO:SOIC-14_3.9x8.7mm_P1.27mm
Changed lines of the file:
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@@
     (property "Reference" "JP9" (id 0) (at 133.35 31.75 0))
     (property "Value" "5v Bus Monitor Disable" (id 1) (at 133.35 34.29 0))
-    (property "Footprint" "" (id 2) (at 133.35 36.83 0)
+    (property "Footprint" "Jumper:SolderJumper-3_P1.3mm_Bridged12_Pad1.0x1.5mm" (id 2) (at 133.35 36.83 0)
       (effects (font (size 1.27 1.27)) hide)
     )
@@
     (property "Reference" "U19" (id 0) (at 226.06 121.92 0))
     (property "Value" "HEF4093B" (id 1) (at 226.06 124.46 0))
-    (property "Footprint" "" (id 2) (at 226.06 130.81 0)
+    (property "Footprint" "Package_SO:SOIC-14_3.9x8.7mm_P1.27mm" (id 2) (at 226.06 130.81 0)
       (effects (font (size 1.27 1.27)) hide)
     )
@@
     (property "Reference" "U19" (id 0) (at 269.24 35.56 0))
     (property "Value" "HEF4093B" (id 1) (at 265.43 45.72 0))
-    (property "Footprint" "" (id 2) (at 265.43 45.72 0)
+    (property "Footprint" "Package_SO:SOIC-14_3.9x8.7mm_P1.27mm" (id 2) (at 265.43 45.72 0)
       (effects (font (size 1.27 1.27)) hide)
     )
@@
     (property "Reference" "U19" (id 0) (at 198.12 50.8 0))
     (property "Value" "HEF4093B" (id 1) (at 198.12 53.34 0))
-    (property "Footprint" "" (id 2) (at 198.12 59.69 0)
+    (property "Footprint" "Package_SO:SOIC-14_3.9x8.7mm_P1.27mm" (id 2) (at 198.12 59.69 0)
       (effects (font (size 1.27 1.27)) hide)
     )
@@
     (property "Reference" "U19" (id 0) (at 224.79 50.8 0))
     (property "Value" "HEF4093B" (id 1) (at 224.79 53.34 0))
-    (property "Footprint" "" (id 2) (at 224.79 59.69 0)
+    (property "Footprint" "Package_SO:SOIC-14_3.9x8.7mm_P1.27mm" (id 2) (at 224.79 59.69 0)
       (effects (font (size 1.27 1.27)) hide)
     )
@@
       (effects (font (size 1.27 1.27)) (justify right))
     )
-    (property "Footprint" "" (id 2) (at 120.65 36.83 0)
+    (property "Footprint" "TestPoint:TestPoint_Pad_D1.5mm" (id 2) (at 120.65 36.83 0)
       (effects (font (size 1.27 1.27)) hide)
     )
@@
     (property "Reference" "U19" (id 0) (at 199.39 121.92 0))
     (property "Value" "HEF4093B" (id 1) (at 199.39 124.46 0))
-    (property "Footprint" "" (id 2) (at 199.39 130.81 0)
+    (property "Footprint" "Package_SO:SOIC-14_3.9x8.7mm_P1.27mm" (id 2) (at 199.39 130.81 0)
       (effects (font (size 1.27 1.27)) hide)
     )
@@
       (effects (font (size 1.27 1.27)) (justify right))
     )
-    (property "Footprint" "" (id 2) (at 121.92 109.22 0)
+    (property "Footprint" "TestPoint:TestPoint_Pad_D1.5mm" (id 2) (at 121.92 109.22 0)
       (effects (font (size 1.27 1.27)) hide)
     )
@@
     (property "Reference" "JP10" (id 0) (at 133.35 106.68 0))
     (property "Value" "12v Bus Monitor Disable" (id 1) (at 133.35 109.22 0))
-    (property "Footprint" "" (id 2) (at 133.35 111.76 0)
-      (effects (font (size 1.27 1.27)) hide)
-    )
+    (property "Footprint" "Jumper:SolderJumper-3_P1.3mm_Bridged12_Pad1.0x1.5mm" (id 2) (at 133.35 111.76 0)
+      (effects (font (size 1.27 1.27)) hide)
+    )

Commit message: Started PCB Layout
Parts:
- removed JP10: 12v Bus Monitor Disable, Jumper:SolderJumper-3_P1.3mm_Bridged12_Pad1.0x1.5mm, symbol 000_Connectors_Immo:Jumper_3_Bridged12
- removed JP9: 5v Bus Monitor Disable, Jumper:SolderJumper-3_P1.3mm_Bridged12_Pad1.0x1.5mm, symbol 000_Connectors_Immo:Jumper_3_Bridged12
- removed R29, R30: 10k, Resistor_SMD:R_0805_2012Metric_Pad1.20x1.40mm_HandSolder, symbol 000_Resistors_Immo:Resistor_0805
Connections:
- net 12V_MON_OUT: now also R28.2, TP9.1, U18.1 (K)
- net 5V_MON_OUT: now also R27.2, TP10.1, U17.1 (K)
- net MCU_5V_IN: no longer TP10.1, TP9.1
Other:
- moved on the sheet: C30, D5, D6, D7, D8, R1a1, R1b1, R27, R28, R2a1, R2b1, R31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
