File: ISOpowerPCB/5to12_logic_v2.kicad_sch (KiCad schematic)
At the start: 25 parts

Commit message: messing around with libraries
Parts:
- gave numbers to parts that had none: 25

Commit message: Started PCB Layout
Parts:
- removed Q14, Q15, Q16, Q17, Q18: BC807, Package_TO_SOT_SMD:SOT-23, symbol Transistor_BJT:BC807
- added Q14, Q15, Q16, Q17, Q18: BC817, Package_TO_SOT_SMD:SOT-23, symbol Transistor_BJT:BC817
- added R35, R36, R37, R38, R39: 10k, Resistor_SMD:R_0805_2012Metric_Pad1.20x1.40mm_HandSolder, symbol 000_Resistors_Immo:Resistor_0805
- R10, R11, R12, R13, R15, R17, R19, R21, R23, R9: value 4k7 -> 10k
- R14, R16, R18, R20, R22: value 22k -> 10k
Connections:
- net 0_OUT: now also Q12.3 (C), R18.1
- net 1_OUT: now also Q13.3 (C), R19.1
- net 2_OUT: now also R20.1, Q14.3 (C)
- net 3_IN: now also R21.1; no longer R12.1
- net 3_OUT: now also Q17.3 (C), R38.1
- net 4_IN: now also R22.1; no longer R13.1
- net 4_OUT: now also Q18.3 (C), R39.1
- net GND: now also Q14.2 (E), Q15.2 (E), Q16.2 (E), Q17.2 (E), Q18.2 (E)
- net HV: now also R12.2, R13.2, R19.2, R23.2, R35.2, R38.2, R39.2; no longer R16.2, R22.2
- net at R17.2: now also Q14.1 (B)
- net at R15.2: now also Q12.1 (B)
- net at Q10.3 (C), R16.1: now also R12.1; no longer R17.1
- net at R21.2: now also Q15.1 (B)
- net at Q13.1 (B): now also R16.2; no longer R13.2
- new net: Q16.3 (C), R35.1, R37.1
- new net: Q18.1 (B), R37.2
- new net: Q11.3 (C), R13.1, R17.1
- new net: Q16.1 (B), R22.2
- new net: Q15.3 (C), R23.1, R36.1
- new net: Q17.1 (B), R36.2
Other:
- moved on the sheet: Q9, R14, R15, R9
