File: ISOpowerPCB/ISOpower_MCU.kicad_sch (KiCad schematic)
At the start: 28 parts, among them J2 ESP_GPIO_B, J3 ESPpin4-7, J4 SDI-SDO, J5 ESP_GPIO_A, J6 prog_power_select, J7 i2c Header, J8 AVR-ISP-6, SW1 SW_Push, U1 ESP32-WROOM-32, U2 AMS1117-3.3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

Commit message: Started PCB Layout
Parts:
- J7: footprint Connector_PinHeader_1.27mm:PinHeader_2x03_P1.27mm_Vertical -> Connector_PinHeader_1.27mm:PinHeader_1x05_P1.27mm_Vertical
Changed lines of the file:
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@@
       (effects (font (size 1.27 1.27)) (justify right))
     )
-    (property "Footprint" "Connector_PinHeader_1.27mm:PinHeader_2x03_P1.27mm_Vertical" (id 2) (at 163.83 177.8 0)
+    (property "Footprint" "Connector_PinHeader_1.27mm:PinHeader_1x05_P1.27mm_Vertical" (id 2) (at 163.83 177.8 0)
       (effects (font (size 1.27 1.27)) hide)
     )

Commit message: PCB Layouts
Parts:
- removed C6: 100n, Capacitor_SMD:C_0805_2012Metric_Pad1.18x1.45mm_HandSolder, symbol 000_Capacitor_Film_Immo:cap_film_0805
- TP6: value TestPoint -> AtMega_Reset
Connections:
- net +5V_IN: no longer C3.1
- net GND: now also C4.2; no longer C4.1
- net MCU_5V_BUS: now also C4.1; no longer R2.1, R3.1
- net +3V3 renamed 3V3_OUT
- net 3V3_OUT: now also C3.1, R2.1, R3.1; no longer C4.2
- net USB_PBUS renamed USB_POUT
Other:
- sheet USB ESP32 CH340 Interface  ports: added none; removed 3V3_IN
- sheet USB MCU CH340 Interface A ports: added none; removed 3V3_IN
- moved on the sheet: C1, C3, C4, L1
