File: ISOpowerPCB/ISOpower_MCU.kicad_sch (KiCad schematic)
At the start: 27 parts, among them J2 ESP_GPIO_B, J3 ESPpin4-7, J4 SDI-SDO, J5 ESP_GPIO_A, J6 prog_power_select, J7 i2c Header, J8 AVR-ISP-6, SW1 SW_Push, U1 ESP32-WROOM-32, U2 AMS1117-3.3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

Commit message: Components placed V1.0
Parts:
- U2: footprint Package_TO_SOT_SMD:TO-252-3_TabPin2 -> Package_TO_SOT_SMD:SOT-223-3_TabPin2
Changed lines of the file:
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@@
     (property "Reference" "U2" (id 0) (at 62.23 55.88 0))
     (property "Value" "AMS1117-3.3" (id 1) (at 62.23 58.42 0))
-    (property "Footprint" "Package_TO_SOT_SMD:TO-252-3_TabPin2" (id 2) (at 62.23 58.42 0)
+    (property "Footprint" "Package_TO_SOT_SMD:SOT-223-3_TabPin2" (id 2) (at 62.23 58.42 0)
       (effects (font (size 1.27 1.27)) hide)
     )
