File: ISOpowerPCB/ch340_ESP32.kicad_sch (KiCad schematic)
At the start: 10 parts, among them J20 USB_B_Mini, Q19 BC817, Q20 BC817, SW2 BOOT, SW3 EN, U14 CH340C

Commit message: PCB Layouts
Connections:
- net 5V_CH340 renamed 5V_IN
Changed lines of the file:
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@@
-    (stroke (width 0) (type default) (color 0 0 0 0))
-  )
-  (wire (pts (xy 25.4 20.32) (xy 36.83 20.32))
     (stroke (width 0) (type default) (color 0 0 0 0))
   )
@@
     (stroke (width 0) (type default) (color 0 0 0 0))
   )
-  (wire (pts (xy 25.4 24.13) (xy 36.83 24.13))
-    (stroke (width 0) (type default) (color 0 0 0 0))
-  )
   (wire (pts (xy 157.48 96.52) (xy 158.75 96.52))
     (stroke (width 0) (type default) (color 0 0 0 0))
@@
   )
   (wire (pts (xy 101.6 80.01) (xy 97.79 80.01))
-    (stroke (width 0) (type default) (color 0 0 0 0))
-  )
-  (wire (pts (xy 25.4 16.51) (xy 36.83 16.51))
     (stroke (width 0) (type default) (color 0 0 0 0))
   )
@@
     (effects (font (size 0.6 0.6)) (justify right bottom))
   )
-  (label "3V3_BUS" (at 26.67 20.32 0)
-    (effects (font (size 1.27 1.27)) (justify left bottom))
-  )
-  (global_label "5V_CH340" (shape output) (at 36.83 16.51 0) (fields_autoplaced)
-    (effects (font (size 1.27 1.27)) (justify left))
-    (property "Intersheet References" "${INTERSHEET_REFS}" (id 0) (at 48.7379 16.4306 0)
-      (effects (font (size 1.27 1.27)) (justify left) hide)
-    )
-  )
-  (global_label "5V_CH340" (shape input) (at 135.89 63.5 90) (fields_autoplaced)
-    (effects (font (size 1.27 1.27)) (justify left))
-    (property "Intersheet References" "${INTERSHEET_REFS}" (id 0) (at 135.9694 51.5921 90)
-      (effects (font (size 1.27 1.27)) (justify right) hide)
-    )
-  )
-  (global_label "3V3_CH340" (shape output) (at 36.83 20.32 0) (fields_autoplaced)
-    (effects (font (size 1.27 1.27)) (justify left))
-    (property "Intersheet References" "${INTERSHEET_REFS}" (id 0) (at 49.9474 20.2406 0)
-      (effects (font (size 1.27 1.27)) (justify left) hide)
-    )
-  )
   (hierarchical_label "RxD_B" (shape input) (at 156.21 80.01 0)
     (effects (font (size 1.27 1.27)) (justify left))
   )
-  (hierarchical_label "3V3_IN" (shape input) (at 25.4 20.32 180)
+  (hierarchical_label "GND" (shape passive) (at 199.39 125.73 270)
     (effects (font (size 1.27 1.27)) (justify right))
   )
@@
     (effects (font (size 1.27 1.27)) (justify left))
   )
-  (hierarchical_label "5V_IN" (shape input) (at 25.4 16.51 180)
-    (effects (font (size 1.27 1.27)) (justify right))
+  (hierarchical_label "GND" (shape passive) (at 116.84 72.39 270)
+    (effects (font (size 1.27 1.27)) (justify right))
+  )
+  (hierarchical_label "5V_IN" (shape input) (at 135.89 63.5 90)
+    (effects (font (size 1.27 1.27)) (justify left))
   )
   (hierarchical_label "USB_VOUT" (shape output) (at 101.6 80.01 0)
     (effects (font (size 1.27 1.27)) (justify left))
   )
-  (hierarchical_label "GND" (shape passive) (at 25.4 24.13 180)
+  (hierarchical_label "GND" (shape passive) (at 199.39 92.71 270)
+    (effects (font (size 1.27 1.27)) (justify right))
+  )
+  (hierarchical_label "GND" (shape passive) (at 135.89 109.22 270)
+    (effects (font (size 1.27 1.27)) (justify right))
+  )
+  (hierarchical_label "GND" (shape passive) (at 90.17 113.03 270)
     (effects (font (size 1.27 1.27)) (justify right))
   )
@@
     (pin "1")
     (pin "2")
-  )
-  (symbol (lib_id "power:GND") (at 199.39 92.71 0) (mirror y) (unit 1)
-    (in_bom yes) (on_board yes) (fields_autoplaced)
-    (property "Reference" "#PWR086" (id 0) (at 199.39 99.06 0)
-      (effects (font (size 1.27 1.27)) hide)
-    )
-    (property "Value" "GND" (id 1) (at 196.85 93.9799 0)
-      (effects (font (size 1.27 1.27)) (justify left))
-    )
-    (property "Footprint" "" (id 2) (at 199.39 92.71 0)
-      (effects (font (size 1.27 1.27)) hide)
-    )
-    (property "Datasheet" "" (id 3) (at 199.39 92.71 0)
-      (effects (font (size 1.27 1.27)) hide)
-    )
-    (pin "1")
-  )
-  (symbol (lib_id "power:GND") (at 116.84 72.39 0) (mirror y) (unit 1)
-    (in_bom yes) (on_board yes) (fields_autoplaced)
-    (property "Reference" "#PWR084" (id 0) (at 116.84 78.74 0)
-      (effects (font (size 1.27 1.27)) hide)
-    )
-    (property "Value" "GND" (id 1) (at 114.3 73.6599 0)
-      (effects (font (size 1.27 1.27)) (justify left))
-    )
-    (property "Footprint" "" (id 2) (at 116.84 72.39 0)
-      (effects (font (size 1.27 1.27)) hide)
-    )
-    (property "Datasheet" "" (id 3) (at 116.84 72.39 0)
-      (effects (font (size 1.27 1.27)) hide)
-    )
-    (pin "1")
   )
   (symbol (lib_id "Interface_USB:CH340C") (at 135.89 87.63 0) (unit 1)
@@
     (pin "9")
   )
-  (symbol (lib_id "power:GND") (at 90.17 113.03 0) (mirror y) (unit 1)
-    (in_bom yes) (on_board yes) (fields_autoplaced)
-    (property "Reference" "#PWR083" (id 0) (at 90.17 119.38 0)
-      (effects (font (size 1.27 1.27)) hide)
-    )
-    (property "Value" "GND" (id 1) (at 87.63 114.2999 0)
-      (effects (font (size 1.27 1.27)) (justify left))
-    )
-    (property "Footprint" "" (id 2) (at 90.17 113.03 0)
-      (effects (font (size 1.27 1.27)) hide)
-    )
-    (property "Datasheet" "" (id 3) (at 90.17 113.03 0)
-      (effects (font (size 1.27 1.27)) hide)
-    )
-    (pin "1")
-  )
   (symbol (lib_id "000_Capacitor_Film_Immo:cap_film_0805") (at 127 71.12 270) (mirror x) (unit 1)
     (in_bom yes) (on_board yes)
@@
     (pin "2")
   )
-  (symbol (lib_id "power:GND") (at 36.83 24.13 90) (unit 1)
-    (in_bom yes) (on_board yes) (fields_autoplaced)
-    (property "Reference" "#PWR082" (id 0) (at 43.18 24.13 0)
-      (effects (font (size 1.27 1.27)) hide)
-    )
-    (property "Value" "GND" (id 1) (at 40.64 24.1299 90)
-      (effects (font (size 1.27 1.27)) (justify right))
-    )
-    (property "Footprint" "" (id 2) (at 36.83 24.13 0)
-      (effects (font (size 1.27 1.27)) hide)
-    )
-    (property "Datasheet" "" (id 3) (at 36.83 24.13 0)
-      (effects (font (size 1.27 1.27)) hide)
-    )
-    (pin "1")
-  )
   (symbol (lib_id "Transistor_BJT:BC817") (at 182.88 88.9 0) (unit 1)
     (in_bom yes) (on_board yes) (fields_autoplaced)
@@
     (pin "1")
     (pin "2")
-  )
-  (symbol (lib_id "power:GND") (at 199.39 125.73 0) (mirror y) (unit 1)
-    (in_bom yes) (on_board yes) (fields_autoplaced)
-    (property "Reference" "#PWR087" (id 0) (at 199.39 132.08 0)
-      (effects (font (size 1.27 1.27)) hide)
-    )
-    (property "Value" "GND" (id 1) (at 196.85 126.9999 0)
-      (effects (font (size 1.27 1.27)) (justify left))
-    )
-    (property "Footprint" "" (id 2) (at 199.39 125.73 0)
-      (effects (font (size 1.27 1.27)) hide)
-    )
-    (property "Datasheet" "" (id 3) (at 199.39 125.73 0)
-      (effects (font (size 1.27 1.27)) hide)
-    )
-    (pin "1")
   )
   (symbol (lib_id "000_Resistors_Immo:Resistor_0805") (at 168.91 88.9 90) (unit 1)
@@
     (pin "2")
   )
-  (symbol (lib_id "power:GND") (at 135.89 109.22 0) (mirror y) (unit 1)
-    (in_bom yes) (on_board yes) (fields_autoplaced)
-    (property "Reference" "#PWR085" (id 0) (at 135.89 115.57 0)
-      (effects (font (size 1.27 1.27)) hide)
-    )
-    (property "Value" "GND" (id 1) (at 133.35 110.4899 0)
-      (effects (font (size 1.27 1.27)) (justify left))
-    )
-    (property "Footprint" "" (id 2) (at 135.89 109.22 0)
-      (effects (font (size 1.27 1.27)) hide)
-    )
-    (property "Datasheet" "" (id 3) (at 135.89 109.22 0)
-      (effects (font (size 1.27 1.27)) hide)
-    )
-    (pin "1")
-  )
   (symbol (lib_id "Transistor_BJT:BC817") (at 182.88 104.14 0) (mirror x) (unit 1)
