File: ISOpowerPCB/logiclevelconverter.kicad_sch (KiCad schematic)
At the start: 5 parts, among them U13 TXS0102DCT

Commit message: PCB Layouts
Changed lines of the file:
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@@
-    (stroke (width 0) (type default) (color 0 0 0 0))
-  )
-  (wire (pts (xy 143.51 113.03) (xy 143.51 116.84))
     (stroke (width 0) (type default) (color 0 0 0 0))
   )
@@
     (stroke (width 0) (type default) (color 0 0 0 0))
   )
-  (wire (pts (xy 22.86 17.78) (xy 27.94 17.78))
-    (stroke (width 0) (type default) (color 0 0 0 0))
-  )
   (wire (pts (xy 146.05 81.28) (xy 146.05 82.55))
     (stroke (width 0) (type default) (color 0 0 0 0))
@@
   )
   (wire (pts (xy 106.68 113.03) (xy 119.38 113.03))
+    (stroke (width 0) (type default) (color 0 0 0 0))
+  )
+  (wire (pts (xy 143.51 113.03) (xy 143.51 116.84))
     (stroke (width 0) (type default) (color 0 0 0 0))
   )
@@
     (effects (font (size 0.8 0.8)) (justify left bottom))
   )
-  (hierarchical_label "GND" (shape passive) (at 22.86 17.78 180)
+  (hierarchical_label "GND" (shape passive) (at 143.51 116.84 270)
     (effects (font (size 1.27 1.27)) (justify right))
   )
@@
     (pin "2")
   )
-  (symbol (lib_id "power:GND") (at 143.51 116.84 0) (unit 1)
-    (in_bom yes) (on_board yes) (fields_autoplaced)
-    (property "Reference" "#PWR081" (id 0) (at 143.51 123.19 0)
-      (effects (font (size 1.27 1.27)) hide)
-    )
-    (property "Value" "GND" (id 1) (at 143.5101 120.65 90)
-      (effects (font (size 1.27 1.27)) (justify right))
-    )
-    (property "Footprint" "" (id 2) (at 143.51 116.84 0)
-      (effects (font (size 1.27 1.27)) hide)
-    )
-    (property "Datasheet" "" (id 3) (at 143.51 116.84 0)
-      (effects (font (size 1.27 1.27)) hide)
-    )
-    (pin "1")
-  )
-  (symbol (lib_id "power:GND") (at 27.94 17.78 90) (unit 1)
-    (in_bom yes) (on_board yes) (fields_autoplaced)
-    (property "Reference" "#PWR080" (id 0) (at 34.29 17.78 0)
-      (effects (font (size 1.27 1.27)) hide)
-    )
-    (property "Value" "GND" (id 1) (at 31.75 17.7799 90)
-      (effects (font (size 1.27 1.27)) (justify right))
-    )
-    (property "Footprint" "" (id 2) (at 27.94 17.78 0)
-      (effects (font (size 1.27 1.27)) hide)
-    )
-    (property "Datasheet" "" (id 3) (at 27.94 17.78 0)
-      (effects (font (size 1.27 1.27)) hide)
-    )
-    (pin "1")
-  )
   (symbol (lib_id "000_Capacitor_Electrolytic_Immo:100u") (at 119.38 107.95 0) (unit 1)

Commit message: Components placed V1.0
Parts:
- removed C31: 100u, Capacitor_SMD:CP_Elec_6.3x7.7, symbol 000_Capacitor_Electrolytic_Immo:100u
- added C6: 100n, Capacitor_SMD:C_0805_2012Metric_Pad1.18x1.45mm_HandSolder, symbol 000_Capacitor_Film_Immo:cap_film_0805
- added R29: 1k, Resistor_SMD:R_0805_2012Metric_Pad1.20x1.40mm_HandSolder, symbol 000_Resistors_Immo:Resistor_0805
Connections:
- net 3V3_IN: now also R29.1; no longer R24.1, U13.6 (OE)
- net GND: now also C6.2
- new net: C6.1, R24.1, R29.2, U13.6 (OE)
Changed lines of the file:
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@@
   (junction (at 119.38 102.87) (diameter 0) (color 0 0 0 0)
-  )
-  (junction (at 119.38 81.28) (diameter 0) (color 0 0 0 0)
   )
   (junction (at 143.51 113.03) (diameter 0) (color 0 0 0 0)
   )
   (junction (at 128.27 113.03) (diameter 0) (color 0 0 0 0)
+  )
+  (junction (at 119.38 81.28) (diameter 0) (color 0 0 0 0)
   )
   (junction (at 128.27 102.87) (diameter 0) (color 0 0 0 0)
@@
     (stroke (width 0) (type default) (color 0 0 0 0))
   )
+  (wire (pts (xy 119.38 87.63) (xy 119.38 81.28))
+    (stroke (width 0) (type default) (color 0 0 0 0))
+  )
   (wire (pts (xy 128.27 102.87) (xy 128.27 104.14))
     (stroke (width 0) (type default) (color 0 0 0 0))
@@
     (stroke (width 0) (type default) (color 0 0 0 0))
   )
-  (wire (pts (xy 140.97 81.28) (xy 119.38 81.28))
-    (stroke (width 0) (type default) (color 0 0 0 0))
-  )
-  (wire (pts (xy 128.27 102.87) (xy 119.38 102.87))
+  (wire (pts (xy 119.38 102.87) (xy 128.27 102.87))
     (stroke (width 0) (type default) (color 0 0 0 0))
   )
   (wire (pts (xy 157.48 92.71) (xy 153.67 92.71))
+    (stroke (width 0) (type default) (color 0 0 0 0))
+  )
+  (wire (pts (xy 119.38 81.28) (xy 140.97 81.28))
     (stroke (width 0) (type default) (color 0 0 0 0))
   )
@@
     (stroke (width 0) (type default) (color 0 0 0 0))
   )
+  (wire (pts (xy 119.38 95.25) (xy 119.38 102.87))
+    (stroke (width 0) (type default) (color 0 0 0 0))
+  )
   (wire (pts (xy 146.05 81.28) (xy 146.05 82.55))
     (stroke (width 0) (type default) (color 0 0 0 0))
@@
     (stroke (width 0) (type default) (color 0 0 0 0))
   )
-  (wire (pts (xy 119.38 81.28) (xy 106.68 81.28))
+  (wire (pts (xy 106.68 81.28) (xy 119.38 81.28))
     (stroke (width 0) (type default) (color 0 0 0 0))
   )
@@
   )
   (wire (pts (xy 140.97 81.28) (xy 140.97 82.55))
-    (stroke (width 0) (type default) (color 0 0 0 0))
-  )
-  (wire (pts (xy 119.38 102.87) (xy 119.38 81.28))
     (stroke (width 0) (type default) (color 0 0 0 0))
   )
@@
     (pin "2")
   )
+  (symbol (lib_id "000_Resistors_Immo:Resistor_0805") (at 119.38 91.44 0) (unit 1)
+    (in_bom yes) (on_board yes) (fields_autoplaced)
+    (property "Reference" "R29" (id 0) (at 121.92 90.1699 0)
+      (effects (font (size 1.27 1.27)) (justify left))
+    )
+    (property "Value" "1k" (id 1) (at 121.92 92.7099 0)
+      (effects (font (size 1.27 1.27)) (justify left))
+    )
+    (property "Footprint" "Resistor_SMD:R_0805_2012Metric_Pad1.20x1.40mm_HandSolder" (id 2) (at 117.602 91.44 90)
+      (effects (font (size 1.27 1.27)) hide)
+    )
+    (property "Datasheet" "~" (id 3) (at 119.38 91.44 0)
+      (effects (font (size 1.27 1.27)) hide)
+    )
+    (pin "1")
+    (pin "2")
+  )
   (symbol (lib_id "000_Capacitor_Film_Immo:cap_film_0805") (at 106.68 96.52 0) (unit 1)
     (in_bom yes) (on_board yes) (fields_autoplaced)
@@
     (pin "2")
   )
-  (symbol (lib_id "000_Capacitor_Electrolytic_Immo:100u") (at 119.38 107.95 0) (unit 1)
-    (in_bom yes) (on_board yes)
-    (property "Reference" "C31" (id 0) (at 113.03 105.41 0)
+  (symbol (lib_id "000_Capacitor_Film_Immo:cap_film_0805") (at 119.38 107.95 0) (unit 1)
+    (in_bom yes) (on_board yes) (fields_autoplaced)
+    (property "Reference" "C6" (id 0) (at 123.19 106.6799 0)
       (effects (font (size 1.27 1.27)) (justify left))
     )
-    (property "Value" "100u" (id 1) (at 111.76 109.22 0)
+    (property "Value" "100n" (id 1) (at 123.19 109.2199 0)
       (effects (font (size 1.27 1.27)) (justify left))
     )
-    (property "Footprint" "Capacitor_SMD:CP_Elec_6.3x7.7" (id 2) (at 120.3452 111.76 0)
+    (property "Footprint" "Capacitor_SMD:C_0805_2012Metric_Pad1.18x1.45mm_HandSolder" (id 2) (at 120.65 118.11 0)
       (effects (font (size 1.27 1.27)) hide)
     )
