File: ISOpowerPCB/ISOpower.kicad_pcb (KiCad board)
At the start: 2 copper layers, 172 parts, among them J1 XT60_connector_DC_60A_male, J10 USB_CH_A, J11 USB_CH_A, J12 USB_CH_A, J13 USB_CH_A, J14 XT30_connector_DC_30A_female, J15 XT30_connector_DC_30A_female, J16 XT30_connector_DC_30A_female, J17 XT30_connector_DC_30A_female, J18 XT30_connector_DC_30A_female, J19 USB_B_Mini, J2 ESP_GPIO_B, J20 USB_B_Mini, J21 24vTerminal, J22 12vTerminal, J23 5vTerminal, J3 ESPpin4-7, J4 SDI-SDO, J5 ESP_GPIO_A, J6 Conn_01x03_Male, J7 i2c Header, J8 AVR-ISP-6, J9 USB_CH_A, M1 Fan_IEC60617, Q1 IRF5305_PBF, Q10 BC817, Q11 BC817, Q12 BC817, Q13 BC817, Q14 BC807, Q15 BC807, Q16 BC807, Q17 BC807, Q18 BC807, Q19 BC817, Q2 IRF5305_PBF, Q20 BC817, Q3 IRF5305_PBF, Q4 IRF5305_PBF, Q5 IRF5305_PBF, Q6 IRF5305_PBF, Q7 IRF5305_PBF, Q8 IRF5305_PBF, Q9 BC817, SW1 SW_Push, SW2 BOOT, SW3 EN, U1 ESP32-WROOM-32, U10 LM2596S-5, U12 CH340C, U13 TXS0102DCT, U14 CH340C, U15 TL431DBZ, U16 TL431DBZ, U17 TL431DBZ, U18 TL431DBZ, U19 HEF4093B, U2 AMS1117-3.3, U3 ATmega328PB-M, U4 i6A4W020A-DC-DC-250W, U5 i6A4W020A-DC-DC-250W, U6 ACS712xLCTR-30A, U7 ACS712xLCTR-30A, Y1 16MHz

Commit message: Started PCB Layout
Parts:
- removed JP10: 12v Bus Monitor Disable, Jumper:SolderJumper-3_P1.3mm_Bridged12_Pad1.0x1.5mm
- removed JP9: 5v Bus Monitor Disable, Jumper:SolderJumper-3_P1.3mm_Bridged12_Pad1.0x1.5mm
- added N1: Net_Tie, NetTie:NetTie-2_SMD_Pad0.5mm, F.Cu at (-66.0, 304.8)
- added N2: Net_Tie, NetTie:NetTie-2_SMD_Pad0.5mm, F.Cu at (-69.1, 304.8)
- added Q10: BC817, Package_TO_SOT_SMD:SOT-23, F.Cu at (-99.6, 310.4)
- added Q11: BC817, Package_TO_SOT_SMD:SOT-23, F.Cu at (-99.6, 306.0)
- added Q12: BC817, Package_TO_SOT_SMD:SOT-23, F.Cu at (-94.7, 306.0)
- added Q13: BC817, Package_TO_SOT_SMD:SOT-23, F.Cu at (-104.5, 306.0)
- added Q14: BC817, Package_TO_SOT_SMD:SOT-23, F.Cu at (-104.5, 310.4)
- added Q15: BC817, Package_TO_SOT_SMD:SOT-23, F.Cu at (-104.5, 319.4)
- added Q16: BC817, Package_TO_SOT_SMD:SOT-23, F.Cu at (-104.5, 314.9)
- added Q17: BC817, Package_TO_SOT_SMD:SOT-23, F.Cu at (-99.6, 314.9)
- added Q18: BC817, Package_TO_SOT_SMD:SOT-23, F.Cu at (-94.7, 310.4)
- added R10: 10k, Resistor_SMD:R_0805_2012Metric_Pad1.20x1.40mm_HandSolder, F.Cu at (-89.9, 311.1)
- added R11: 10k, Resistor_SMD:R_0805_2012Metric_Pad1.20x1.40mm_HandSolder, F.Cu at (-89.9, 305.2)
- added R12: 10k, Resistor_SMD:R_0805_2012Metric_Pad1.20x1.40mm_HandSolder, F.Cu at (-90.0, 317.1)
- added R13: 10k, Resistor_SMD:R_0805_2012Metric_Pad1.20x1.40mm_HandSolder, F.Cu at (-90.2, 320.1)
- added R16: 10k, Resistor_SMD:R_0805_2012Metric_Pad1.20x1.40mm_HandSolder, F.Cu at (-85.1, 308.2)
- added R17: 10k, Resistor_SMD:R_0805_2012Metric_Pad1.20x1.40mm_HandSolder, F.Cu at (-94.8, 314.1)
- added R18: 10k, Resistor_SMD:R_0805_2012Metric_Pad1.20x1.40mm_HandSolder, F.Cu at (-80.4, 305.2)
- added R19: 10k, Resistor_SMD:R_0805_2012Metric_Pad1.20x1.40mm_HandSolder, F.Cu at (-85.1, 311.1)
- added R20: 10k, Resistor_SMD:R_0805_2012Metric_Pad1.20x1.40mm_HandSolder, F.Cu at (-94.9, 320.1)
- added R21: 10k, Resistor_SMD:R_0805_2012Metric_Pad1.20x1.40mm_HandSolder, F.Cu at (-99.7, 318.6)
- added R22: 10k, Resistor_SMD:R_0805_2012Metric_Pad1.20x1.40mm_HandSolder, F.Cu at (-80.4, 308.2)
- added R23: 10k, Resistor_SMD:R_0805_2012Metric_Pad1.20x1.40mm_HandSolder, F.Cu at (-80.4, 311.1)
- added R35: 10k, Resistor_SMD:R_0805_2012Metric_Pad1.20x1.40mm_HandSolder, F.Cu at (-85.3, 314.1)
- added R36: 10k, Resistor_SMD:R_0805_2012Metric_Pad1.20x1.40mm_HandSolder, F.Cu at (-90.0, 314.1)
- added R37: 10k, Resistor_SMD:R_0805_2012Metric_Pad1.20x1.40mm_HandSolder, F.Cu at (-89.9, 308.2)
- added R38: 10k, Resistor_SMD:R_0805_2012Metric_Pad1.20x1.40mm_HandSolder, F.Cu at (-94.8, 317.1)
- added R39: 10k, Resistor_SMD:R_0805_2012Metric_Pad1.20x1.40mm_HandSolder, F.Cu at (-85.1, 305.2)
- J6: value Conn_01x03_Male -> prog_power_select
- JP1: value Jumper_3_Bridged12 -> prog_power_select
- R14: value 22k -> 10k
- R15, R9: value 4k7 -> 10k
- moved C30 355.1 mm to (228.6, -24.1), turned to 180 degrees
- moved D8 350.6 mm to (236.2, -16.9), turned to 180 degrees
- moved R34 347.9 mm to (240.3, -16.5)
- moved R31 340.8 mm to (222.5, -21.6)
- moved R32 339.6 mm to (240.3, -19.1)
- moved D5 328.6 mm to (223.3, -19.1)
- moved R33 326.4 mm to (223.2, -15.0)
- moved H1 322.9 mm to (91.4, 147.3)
- moved D7 320.2 mm to (223.3, -17.0)
- moved C31 304.1 mm to (227.3, 157.5)
- moved Q2 301.7 mm to (141.7, 83.8)
- moved JP1 293.1 mm to (172.7, 112.1)
- moved Q7 284.9 mm to (160.7, 70.9), turned to 180 degrees
- moved H4 281.1 mm to (91.4, 58.4)
- moved J22 274.3 mm to (91.4, 68.6), turned to -90 degrees
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Connections:
- net Net-(C11-Pad1) renamed /Power Distribution/5V_I_SENSE_IP
- net Net-(C12-Pad1) renamed /Power Distribution/12V_I_SENSE_IP
- net Net-(F1-Pad1) renamed /24V_0
- net Net-(F1-Pad2) renamed /24V_1
- net Net-(J14-Pad2) renamed /Power Outputs/12V_OP_0
- net Net-(J15-Pad2) renamed /Power Outputs/12V_OP_1
- net Net-(J16-Pad2) renamed /Power Outputs/12V_OP_2
- net Net-(J17-Pad2) renamed /Power Outputs/12V_OP_3
- net Net-(J18-Pad2) renamed /Power Outputs/12V_OP_4
- C2 pad 1: MCU_5V -> MCU_5V_BUS
- C23 pad 1: MCU_5V -> MCU_5V_BUS
- C27 pad 1: MCU_5V -> MCU_5V_BUS
- C28 pad 1: MCU_5V -> MCU_5V_BUS
- C6 pad 2: MCU_5V -> MCU_5V_BUS
- D4 pad 4: MCU_5V -> MCU_5V_BUS
- J6 pad 2: MCU_5V -> MCU_5V_BUS
- J7 pad 3: MCU_5V -> MCU_5V_BUS
- J8 pad 2: MCU_5V -> MCU_5V_BUS
- JP1 pad 2: MCU_5V -> MCU_5V_BUS
- L1 pad 1: MCU_5V -> MCU_5V_BUS
- R15 pad 2: Net-(Q14-Pad1) -> Net-(R15-Pad2)
- R2 pad 1: MCU_5V -> MCU_5V_BUS
- R27 pad 2: Net-(R27-Pad2) -> /5V_BUS_MONITOR
- R28 pad 2: Net-(R28-Pad2) -> /12V_BUS_MONITOR
- R3 pad 1: MCU_5V -> MCU_5V_BUS
- R5 pad 1: MCU_5V -> MCU_5V_BUS
- TP10 pad 1: MCU_5V -> /5V_BUS_MONITOR
- TP9 pad 1: MCU_5V -> /12V_BUS_MONITOR
- U12 pad 16: MCU_5V -> MCU_5V_BUS
- U13 pad 7: MCU_5V -> MCU_5V_BUS
- U14 pad 16: MCU_5V -> MCU_5V_BUS
- U17 pad 1: Net-(R27-Pad2) -> /5V_BUS_MONITOR
- U18 pad 1: Net-(R28-Pad2) -> /12V_BUS_MONITOR
- U2 pad 3: MCU_5V -> MCU_5V_BUS
- U3 pad 18: MCU_5V -> MCU_5V_BUS
- U3 pad 4: MCU_5V -> MCU_5V_BUS
- U6 pad 3: +5V_BUS -> /Power Distribution/5V_I_SENSE_OP
- U6 pad 4: +5V_BUS -> /Power Distribution/5V_I_SENSE_OP
- U7 pad 3: +12V_BUS -> /Power Distribution/12V_I_SENSE_OP
- U7 pad 4: +12V_BUS -> /Power Distribution/12V_I_SENSE_OP
Other:
- board outline added: 119.4 x 99.1 mm

Commit message: PCB Layouts
Parts:
- removed C6: 100n, Capacitor_SMD:C_0805_2012Metric_Pad1.18x1.45mm_HandSolder
- removed the Q10 at (238.4, 233.1)
- removed the Q11 at (248.7, 243.8)
- removed the Q12 at (251.5, 231.1)
- removed the Q13 at (238.4, 223.5)
- removed the Q14 at (233.5, 228.6)
- removed the Q15 at (223.5, 221.0)
- removed the Q16 at (259.1, 243.8)
- removed the Q17 at (233.5, 233.1)
- removed the Q18 at (228.6, 233.1)
- removed the R10 at (228.4, 285.3)
- removed the R11 at (223.5, 289.8)
- removed the R12 at (208.8, 312.3)
- removed the R13 at (223.3, 292.7)
- removed the R16 at (213.7, 295.7)
- removed the R17 at (233.1, 282.4)
- removed the R18 at (213.6, 300.2)
- removed the R19 at (213.6, 303.1)
- removed the R20 at (208.8, 300.2)
- removed the R21 at (223.5, 286.8)
- removed the R22 at (228.4, 282.4)
- removed the R23 at (218.4, 297.2)
- removed R29, R30: 10k, Resistor_SMD:R_0805_2012Metric_Pad1.20x1.40mm_HandSolder
- added J24: dio_spare, Connector_PinHeader_1.27mm:PinHeader_1x01_P1.27mm_Vertical, F.Cu at (94.0, 102.9)
- added J25: adc_spare, Connector_PinHeader_1.27mm:PinHeader_1x02_P1.27mm_Vertical, F.Cu at (94.0, 66.0)
- added J26: USB_5v, Connector_PinHeader_1.27mm:PinHeader_1x01_P1.27mm_Vertical, F.Cu at (139.7, 68.6)
- added J27: pwr_ctls, Connector_PinSocket_1.27mm:PinSocket_1x05_P1.27mm_Vertical, F.Cu at (94.0, 94.0)
- added J28: MCU_DIO_A, Connector_PinHeader_1.27mm:PinHeader_1x05_P1.27mm_Vertical, F.Cu at (273.1, 41.9)
- added J29: sensor_op, Connector_PinSocket_1.27mm:PinSocket_1x04_P1.27mm_Vertical, F.Cu at (94.0, 70.5)
- added J30: MCU_ADC, Connector_PinHeader_1.27mm:PinHeader_1x04_P1.27mm_Vertical, F.Cu at (254.0, 48.3)
- added J31: main_pwr, Connector_PinSocket_1.27mm:PinSocket_1x05_P1.27mm_Vertical, F.Cu at (125.7, 76.2)
- added J32: MCU_PWR, Connector_PinHeader_1.27mm:PinHeader_1x05_P1.27mm_Vertical, F.Cu at (219.9, 115.6)
- added J33: MCU_DIO_B, Connector_PinHeader_1.27mm:PinHeader_1x05_P1.27mm_Vertical, F.Cu at (262.9, 41.9)
- added J34: O/P_ctls, Connector_PinSocket_1.27mm:PinSocket_1x05_P1.27mm_Vertical, F.Cu at (127.0, 97.8)
- JP4: value CH_A_BYPASS -> OP_0
- JP5: value CH_A_BYPASS -> OP_1
- JP6: value CH_A_BYPASS -> OP_2
- JP7: value CH_A_BYPASS -> OP_3
- JP8: value CH_A_BYPASS -> OP_4
- TP6: value TestPoint -> AtMega_Reset
- moved C26 456.6 mm to (361.6, 38.1)
- moved R24 440.3 mm to (354.0, 41.9)
- moved C27 439.2 mm to (361.1, 41.9)
- moved R32 365.0 mm to (-36.8, 218.4)
- moved D6 360.2 mm to (-36.8, 215.9), turned to 0 degrees
- moved R34 358.4 mm to (-36.8, 210.8)
- moved C30 357.7 mm to (-32.3, 220.6), turned to 0 degrees
- moved D8 357.2 mm to (-36.8, 213.4), turned to 0 degrees
- moved U19 349.0 mm to (-30.5, 214.6), turned to 180 degrees
- moved R31 344.2 mm to (-24.1, 218.4), turned to 180 degrees
- moved D5 341.2 mm to (-24.1, 215.9), turned to 180 degrees
- moved D7 338.1 mm to (-24.1, 213.4), turned to 180 degrees
- moved R33 334.9 mm to (-24.1, 210.8), turned to 180 degrees
- moved Q16 324.7 mm to (108.0, 69.3), turned to 180 degrees
- moved Q15 321.5 mm to (108.0, 78.1), turned to 180 degrees
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Connections:
- net +12V_BUS renamed 12V_BUS
- net +5V_BUS renamed 5V_BUS
- net USB_PBUS renamed /MCU/USB_PBUS
- C1 pad 2: GND -> /MCU/GND
- C2 pad 1: MCU_5V_BUS -> /MCU/MCU_5V_BUS
- C2 pad 2: GND -> /MCU/GND
- C23 pad 1: MCU_5V_BUS -> /MCU/MCU_5V_BUS
- C23 pad 2: GND -> /MCU/GND
- C24 pad 2: GND -> /MCU/GND
- C25 pad 1: GND -> /MCU/GND
- C26 pad 1: 3V3_CH340 -> /MCU/3V3_BUS
- C26 pad 2: GND -> /MCU/GND
- C27 pad 1: MCU_5V_BUS -> /MCU/MCU_5V_BUS
- C27 pad 2: GND -> /MCU/GND
- C28 pad 1: MCU_5V_BUS -> /MCU/MCU_5V_BUS
- C28 pad 2: GND -> /MCU/GND
- C29 pad 2: GND -> /MCU/GND
- C3 pad 1: MCU_5V -> /MCU/3V3_BUS
- C3 pad 2: GND -> /MCU/GND
- C31 pad 1: 3V3_CH340 -> /MCU/3V3_BUS
- C31 pad 2: GND -> /MCU/GND
- C4 pad 1: GND -> /MCU/MCU_5V_BUS
- C4 pad 2: 3V3_CH340 -> /MCU/GND
- C5 pad 1: 3V3_CH340 -> /MCU/3V3_BUS
- C5 pad 2: GND -> /MCU/GND
- C7 pad 2: GND -> /MCU/GND
- C8 pad 2: GND -> /MCU/GND
- D4 pad 4: MCU_5V_BUS -> /MCU/MCU_5V_BUS
- D7 pad 2: Net-(D7-Pad2) -> Net-(U19-Pad4)
- J19 pad 5: GND -> /MCU/GND
- J20 pad 5: GND -> /MCU/GND
- J20 pad 6: GND -> /MCU/GND
- J6 pad 2: MCU_5V_BUS -> /MCU/MCU_5V_BUS
- J6 pad 3: MCU_5V -> /MCU/+5V_IN
- J7 pad 1: GND -> /MCU/GND
- J7 pad 2: 3V3_CH340 -> /MCU/3V3_BUS
- J7 pad 3: MCU_5V_BUS -> /MCU/MCU_5V_BUS
- J8 pad 2: MCU_5V_BUS -> /MCU/MCU_5V_BUS
- J8 pad 6: GND -> /MCU/GND
- JP1 pad 1: MCU_5V -> /MCU/+5V_IN
- JP1 pad 2: MCU_5V_BUS -> /MCU/MCU_5V_BUS
- L1 pad 1: MCU_5V_BUS -> /MCU/MCU_5V_BUS
- L1 pad 2: GND -> /MCU/GND
- R10 pad 1: /MCU/CH_G -> /Power Outputs/CH_G_CTRL
- R11 pad 1: /MCU/CH_H -> /Power Outputs/CH_H_CTRL
- R2 pad 1: MCU_5V_BUS -> /MCU/3V3_BUS
- R21 pad 1: /MCU/CH_I -> /Power Outputs/CH_I_CTRL
- R22 pad 1: /MCU/CH_J -> /Power Outputs/CH_J_CTRL
- R24 pad 1: 3V3_CH340 -> /MCU/3V3_BUS
- R24 pad 2: GND -> /MCU/GND
- R3 pad 1: MCU_5V_BUS -> /MCU/3V3_BUS
- R4 pad 2: GND -> /MCU/GND
- R5 pad 1: MCU_5V_BUS -> /MCU/MCU_5V_BUS
- R8 pad 2: GND -> /MCU/GND
- R9 pad 1: /MCU/CH_F -> /Power Outputs/CH_F_CTRL
- SW1 pad 2: GND -> /MCU/GND
- SW2 pad 2: GND -> /MCU/GND
- SW3 pad 2: GND -> /MCU/GND
- TP3 pad 1: 3V3_CH340 -> /3V3_BUS
- U1 pad 1: GND -> /MCU/GND
- U1 pad 15: GND -> /MCU/GND
- U1 pad 2: 3V3_CH340 -> /MCU/3V3_BUS
- U1 pad 38: GND -> /MCU/GND
- U1 pad 39: GND -> /MCU/GND
- U12 pad 1: GND -> /MCU/GND
- U12 pad 16: MCU_5V_BUS -> /MCU/MCU_5V_BUS
- U13 pad 2: GND -> /MCU/GND
- U13 pad 3: 3V3_CH340 -> /MCU/3V3_BUS
- U13 pad 6: 3V3_CH340 -> /MCU/3V3_BUS
- U13 pad 7: MCU_5V_BUS -> /MCU/MCU_5V_BUS
- U14 pad 1: GND -> /MCU/GND
- U14 pad 16: MCU_5V_BUS -> /MCU/MCU_5V_BUS
- U19 pad 10: Net-(D7-Pad2) -> Net-(D6-Pad2)
- U19 pad 4: Net-(D6-Pad2) -> Net-(U19-Pad4)
- U19 pad 5: /12V_BUS_MONITOR -> Net-(D5-Pad2)
- U19 pad 6: /12V_BUS_MONITOR -> Net-(D5-Pad2)
- U19 pad 8: Net-(D5-Pad2) -> Net-(U19-Pad8)
- U19 pad 9: Net-(D5-Pad2) -> Net-(U19-Pad8)
- U2 pad 1: GND -> /MCU/GND
- U2 pad 2: 3V3_CH340 -> /MCU/3V3_BUS
- U2 pad 3: MCU_5V_BUS -> /MCU/MCU_5V_BUS
- U3 pad 1: /BUS_B_DISABLE -> /MCU/CH_B
- U3 pad 10: /12V_BUS_MONITOR -> /MCU/IN_E
- U3 pad 18: MCU_5V_BUS -> /MCU/MCU_5V_BUS
- U3 pad 19: /BUS_I_SENSE_A -> /MCU/ADC6
- U3 pad 21: GND -> /MCU/GND
- U3 pad 22: /BUS_I_SENSE_B -> /MCU/ADC7
- U3 pad 32: /BUS_A_DISABLE -> /MCU/CH_A
- U3 pad 33: GND -> /MCU/GND
- U3 pad 4: MCU_5V_BUS -> /MCU/MCU_5V_BUS
- U3 pad 5: GND -> /MCU/GND
- U3 pad 9: /5V_BUS_MONITOR -> /MCU/IN_D
Other:
- copper layers 2 -> 4

Commit message: Components placed V1.0
Parts:
- removed C31: 100u, Capacitor_SMD:CP_Elec_6.3x7.7
- removed J27: pwr_ctls, Connector_PinSocket_1.27mm:PinSocket_1x05_P1.27mm_Vertical
- removed J28: MCU_DIO_A, Connector_PinHeader_1.27mm:PinHeader_1x05_P1.27mm_Vertical
- removed J32: MCU_PWR, Connector_PinHeader_1.27mm:PinHeader_1x05_P1.27mm_Vertical
- removed J33: MCU_DIO_B, Connector_PinHeader_1.27mm:PinHeader_1x05_P1.27mm_Vertical
- removed J34: O/P_ctls, Connector_PinSocket_1.27mm:PinSocket_1x05_P1.27mm_Vertical
- removed U12: CH340C, Package_SO:SOIC-16_3.9x9.9mm_P1.27mm
- added C6: 100n, Capacitor_SMD:C_0805_2012Metric_Pad1.18x1.45mm_HandSolder, F.Cu at (242.6, 107.1)
- added D9: Blue, LED_SMD:LED_0805_2012Metric_Pad1.15x1.40mm_HandSolder, F.Cu at (241.5, 98.4)
- added H10: MountingHole, MountingHole:MountingHole_3.2mm_M3, F.Cu at (255.3, 106.0)
- added H5: MountingHole, MountingHole:MountingHole_3.2mm_M3, F.Cu at (255.3, 79.4)
- added H6: MountingHole, MountingHole:MountingHole_3.2mm_M3, F.Cu at (216.5, 79.4)
- added H7: MountingHole, MountingHole:MountingHole_3.2mm_M3, F.Cu at (96.5, 82.5)
- added H8: MountingHole, MountingHole:MountingHole_3.2mm_M3, F.Cu at (135.3, 109.2)
- added H9: MountingHole, MountingHole:MountingHole_3.2mm_M3, F.Cu at (135.3, 82.5)
- added R29: 1k, Resistor_SMD:R_0805_2012Metric_Pad1.20x1.40mm_HandSolder, F.Cu at (241.7, 103.5)
- added R30: 330r, Resistor_SMD:R_0805_2012Metric_Pad1.20x1.40mm_HandSolder, F.Cu at (241.6, 101.0)
- added U8: CH340C, Package_SO:SOIC-16_3.9x9.9mm_P1.27mm, F.Cu at (121.9, 108.6)
- J1: footprint Connector_AMASS:AMASS_XT60-M_1x02_P7.20mm_Vertical -> Connector_AMASS:AMASS_XT60PW-M
- J19: value USB_B_Mini -> ESP32_header; footprint Connector_USB:USB_Mini-B_Lumberg_2486_01_Horizontal -> Connector_PinHeader_1.27mm:PinHeader_1x10_P1.27mm_Vertical; moved to B.Cu
- J29: value sensor_op -> wifi_header; footprint Connector_PinSocket_1.27mm:PinSocket_1x04_P1.27mm_Vertical -> Connector_PinSocket_1.27mm:PinSocket_1x10_P1.27mm_Vertical
- J30: value MCU_ADC -> 3V3_spare; footprint Connector_PinHeader_1.27mm:PinHeader_1x04_P1.27mm_Vertical -> Connector_PinHeader_1.27mm:PinHeader_1x01_P1.27mm_Vertical
- J31: value main_pwr -> USB_B_Mini; footprint Connector_PinSocket_1.27mm:PinSocket_1x05_P1.27mm_Vertical -> Connector_USB:USB_Mini-B_Lumberg_2486_01_Horizontal
- R4: value 10k -> 330r
- U2: footprint Package_TO_SOT_SMD:TO-252-3_TabPin2 -> Package_TO_SOT_SMD:SOT-223-3_TabPin2
- moved TP9 324.1 mm to (85.1, 97.2)
- moved TP10 323.2 mm to (88.3, 97.2)
- moved TP4 314.2 mm to (116.8, 31.8)
- moved TP1 303.6 mm to (116.8, 26.7)
- moved TP3 299.6 mm to (80.0, 106.0)
- moved TP2 291.0 mm to (130.8, 26.7)
- moved TP5 253.8 mm to (113.0, 116.8)
- moved TP6 248.3 mm to (140.3, 113.0)
- moved TP8 244.5 mm to (129.5, 100.3)
- moved TP7 240.8 mm to (140.3, 107.3)
- moved R32 204.2 mm to (33.4, 26.7), turned to 180 degrees
- moved D6 199.5 mm to (33.4, 29.2), turned to 180 degrees
- moved D8 194.7 mm to (33.4, 31.8), turned to 180 degrees
- moved C24 194.0 mm to (113.9, 113.0), turned to 180 degrees
- moved R2a1 192.1 mm to (97.8, 96.5)
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Connections:
- net /MCU/Logic Level Conversion/0A renamed /ESP32_Daughterboard/Logic Level Conversion/0A
- net /MCU/Logic Level Conversion/1A renamed /ESP32_Daughterboard/Logic Level Conversion/1A
- net /MCU/USB ESP32 CH340 Interface /ESP_EN renamed /ESP32_Daughterboard/USB ESP32 CH340 Interface /ESP_EN
- net /MCU/USB ESP32 CH340 Interface /ESP_IO0 renamed /ESP32_Daughterboard/USB ESP32 CH340 Interface /ESP_IO0
- net /MCU/USB ESP32 CH340 Interface /RxD_B renamed /ESP32_Daughterboard/USB ESP32 CH340 Interface /RxD_B
- net /MCU/USB ESP32 CH340 Interface /TxD_B renamed /ESP32_Daughterboard/USB ESP32 CH340 Interface /TxD_B
- net /MCU/USB MCU CH340 Interface A/DTR_A renamed /AtMega328p/USB MCU CH340 Interface A/DTR_A
- C1 pad 2: /MCU/GND -> /ESP32_Daughterboard/GND
- C2 pad 1: /MCU/MCU_5V_BUS -> /ESP32_Daughterboard/MCU_5V_BUS
- C2 pad 2: /MCU/GND -> /ESP32_Daughterboard/GND
- C23 pad 1: /MCU/MCU_5V_BUS -> /AtMega328p/MCU_5V_BUS
- C23 pad 2: /MCU/GND -> GND
- C24 pad 2: /MCU/GND -> GND
- C25 pad 1: /MCU/GND -> GND
- C26 pad 1: /MCU/3V3_BUS -> /ESP32_Daughterboard/3V3_BUS
- C26 pad 2: /MCU/GND -> /ESP32_Daughterboard/GND
- C27 pad 1: /MCU/MCU_5V_BUS -> /ESP32_Daughterboard/MCU_5V_BUS
- C27 pad 2: /MCU/GND -> /ESP32_Daughterboard/GND
- C28 pad 1: /MCU/MCU_5V_BUS -> /ESP32_Daughterboard/MCU_5V_BUS
- C28 pad 2: /MCU/GND -> /ESP32_Daughterboard/GND
- C29 pad 2: /MCU/GND -> /ESP32_Daughterboard/GND
- C3 pad 1: /MCU/3V3_BUS -> /ESP32_Daughterboard/3V3_BUS
- C3 pad 2: /MCU/GND -> /ESP32_Daughterboard/GND
- C4 pad 1: /MCU/MCU_5V_BUS -> /AtMega328p/MCU_5V_BUS
- C4 pad 2: /MCU/GND -> GND
- C5 pad 1: /MCU/3V3_BUS -> /ESP32_Daughterboard/3V3_BUS
- C5 pad 2: /MCU/GND -> /ESP32_Daughterboard/GND
- C7 pad 2: /MCU/GND -> GND
- C8 pad 2: /MCU/GND -> GND
- D4 pad 4: /MCU/MCU_5V_BUS -> /AtMega328p/MCU_5V_BUS
- J19 pad 1: /MCU/USB_PBUS -> /ESP32_Daughterboard/GND
- J19 pad 2: Net-(D4-Pad2) -> /ESP32_Daughterboard/3V3_BUS
- J19 pad 3: Net-(D4-Pad3) -> /ESP32_Daughterboard/MCU_5V_BUS
- J19 pad 4: unconnected-(J19-Pad4) -> /ESP32_Daughterboard/USB_PBUS
- J19 pad 5: /MCU/GND -> unconnected-(J19-Pad5)
- J19 pad 6: Net-(C25-Pad2) -> unconnected-(J19-Pad6)
- J20 pad 1: /MCU/USB_PBUS -> /ESP32_Daughterboard/USB_PBUS
- J20 pad 5: /MCU/GND -> /ESP32_Daughterboard/GND
- J20 pad 6: /MCU/GND -> /ESP32_Daughterboard/GND
- J24 pad 1: Net-(J24-Pad1) -> /AtMega328p/CH_C
- J25 pad 1: Net-(J25-Pad1) -> /AtMega328p/ADC5
- J25 pad 2: Net-(J25-Pad2) -> /AtMega328p/ADC4
- J26 pad 1: Net-(J31-Pad4) -> /USB_PBUS
- J29 pad 1: /BUS_I_SENSE_A -> GND
- J29 pad 2: /BUS_I_SENSE_B -> /3V3_BUS
- J29 pad 3: Net-(J25-Pad1) -> /AtMega328p/MCU_5V_BUS
- J29 pad 4: Net-(J25-Pad2) -> /USB_PBUS
- J30 pad 1: /MCU/ADC7 -> /3V3_BUS
- J31 pad 1: GND -> /USB_PBUS
- J31 pad 2: /3V3_BUS -> Net-(D4-Pad2)
- J31 pad 3: MCU_5V -> Net-(D4-Pad3)
- J31 pad 4: Net-(J31-Pad4) -> unconnected-(J31-Pad4)
- J31 pad 5: unconnected-(J31-Pad5) -> GND
- J6 pad 1: /MCU/USB_PBUS -> /USB_PBUS
- J6 pad 2: /MCU/MCU_5V_BUS -> /AtMega328p/MCU_5V_BUS
- J6 pad 3: /MCU/+5V_IN -> MCU_5V
- J7 pad 1: /MCU/GND -> /ESP32_Daughterboard/GND
- J7 pad 2: /MCU/3V3_BUS -> /ESP32_Daughterboard/3V3_BUS
- J7 pad 3: /MCU/MCU_5V_BUS -> /ESP32_Daughterboard/MCU_5V_BUS
- J8 pad 2: /MCU/MCU_5V_BUS -> /AtMega328p/MCU_5V_BUS
- J8 pad 6: /MCU/GND -> GND
- JP1 pad 1: /MCU/+5V_IN -> MCU_5V
- JP1 pad 2: /MCU/MCU_5V_BUS -> /AtMega328p/MCU_5V_BUS
- JP1 pad 3: /MCU/USB_PBUS -> /USB_PBUS
- L1 pad 1: /MCU/MCU_5V_BUS -> /AtMega328p/MCU_5V_BUS
- L1 pad 2: /MCU/GND -> GND
- R10 pad 1: /Power Outputs/CH_G_CTRL -> /AtMega328p/CH_G
- R11 pad 1: /Power Outputs/CH_H_CTRL -> /AtMega328p/CH_H
- R2 pad 1: /MCU/3V3_BUS -> /ESP32_Daughterboard/3V3_BUS
- R21 pad 1: /Power Outputs/CH_I_CTRL -> /AtMega328p/CH_I
- R22 pad 1: /Power Outputs/CH_J_CTRL -> /AtMega328p/CH_J
- R24 pad 1: /MCU/3V3_BUS -> Net-(C6-Pad1)
- R24 pad 2: /MCU/GND -> /ESP32_Daughterboard/GND
- R3 pad 1: /MCU/3V3_BUS -> /ESP32_Daughterboard/3V3_BUS
- R4 pad 2: /MCU/GND -> GND
- R5 pad 1: /MCU/MCU_5V_BUS -> /AtMega328p/MCU_5V_BUS
- R8 pad 2: /MCU/GND -> GND
- R9 pad 1: /Power Outputs/CH_F_CTRL -> /AtMega328p/CH_F
- SW1 pad 2: /MCU/GND -> GND
- SW2 pad 2: /MCU/GND -> /ESP32_Daughterboard/GND
- SW3 pad 2: /MCU/GND -> /ESP32_Daughterboard/GND
- U1 pad 1: /MCU/GND -> /ESP32_Daughterboard/GND
- U1 pad 15: /MCU/GND -> /ESP32_Daughterboard/GND
- U1 pad 2: /MCU/3V3_BUS -> /ESP32_Daughterboard/3V3_BUS
- U1 pad 38: /MCU/GND -> /ESP32_Daughterboard/GND
- U1 pad 39: /MCU/GND -> /ESP32_Daughterboard/GND
- U13 pad 1: SSERIAL_TX -> /ESP32_Daughterboard/SSERIAL_TX
- U13 pad 2: /MCU/GND -> /ESP32_Daughterboard/GND
- U13 pad 3: /MCU/3V3_BUS -> /ESP32_Daughterboard/3V3_BUS
- U13 pad 6: /MCU/3V3_BUS -> Net-(C6-Pad1)
- U13 pad 7: /MCU/MCU_5V_BUS -> /ESP32_Daughterboard/MCU_5V_BUS
- U13 pad 8: SSERIAL_RX -> /ESP32_Daughterboard/SSERIAL_RX
- U14 pad 1: /MCU/GND -> /ESP32_Daughterboard/GND
- U14 pad 16: /MCU/MCU_5V_BUS -> /ESP32_Daughterboard/MCU_5V_BUS
- U19 pad 8: Net-(U19-Pad8) -> /12V_BUS_MONITOR
- U19 pad 9: Net-(U19-Pad8) -> /12V_BUS_MONITOR
- U2 pad 1: /MCU/GND -> /ESP32_Daughterboard/GND
- U2 pad 2: /MCU/3V3_BUS -> /ESP32_Daughterboard/3V3_BUS
- U2 pad 3: /MCU/MCU_5V_BUS -> /ESP32_Daughterboard/MCU_5V_BUS
- U3 pad 1: /MCU/CH_B -> /BUS_B_DISABLE
- U3 pad 10: /MCU/IN_E -> /12V_BUS_MONITOR
- U3 pad 12: SSERIAL_TX -> /AtMega328p/SSERIAL_TX
- U3 pad 13: SSERIAL_RX -> /AtMega328p/SSERIAL_RX
- U3 pad 14: /MCU/CH_F -> /AtMega328p/CH_F
- U3 pad 18: /MCU/MCU_5V_BUS -> /AtMega328p/MCU_5V_BUS
- U3 pad 19: /MCU/ADC6 -> /BUS_I_SENSE_B
- U3 pad 2: /MCU/CH_C -> /AtMega328p/CH_C
- U3 pad 21: /MCU/GND -> GND
- U3 pad 22: /MCU/ADC7 -> /BUS_I_SENSE_A
- U3 pad 23: /MCU/CH_G -> /AtMega328p/CH_G
- U3 pad 24: /MCU/CH_H -> /AtMega328p/CH_H
- U3 pad 25: /MCU/CH_I -> /AtMega328p/CH_I
- U3 pad 26: /MCU/CH_J -> /AtMega328p/CH_J
- U3 pad 27: /MCU/ADC4 -> /AtMega328p/ADC4
- U3 pad 28: /MCU/ADC5 -> /AtMega328p/ADC5
- U3 pad 30: /MCU/USB MCU CH340 Interface A/RxD_A -> /AtMega328p/USB MCU CH340 Interface A/RxD_A
- U3 pad 31: /MCU/USB MCU CH340 Interface A/TxD_A -> /AtMega328p/USB MCU CH340 Interface A/TxD_A
- U3 pad 32: /MCU/CH_A -> /BUS_A_DISABLE
- U3 pad 33: /MCU/GND -> GND
- U3 pad 4: /MCU/MCU_5V_BUS -> /AtMega328p/MCU_5V_BUS
- U3 pad 5: /MCU/GND -> GND
- U3 pad 9: /MCU/IN_D -> /5V_BUS_MONITOR
Other:
- board size 119.4 x 99.1 mm -> 241.8 x 99.1 mm

Commit message: Started Routing V1
Parts:
- Q2, Q3: value IRF5305_PBF -> Si2319CDS; footprint Package_TO_SOT_SMD:TO-263-2 -> Package_TO_SOT_SMD:SOT-23
- R6, R7: footprint Resistor_THT:R_Axial_DIN0309_L9.0mm_D3.2mm_P12.70mm_Horizontal -> Resistor_THT:R_Axial_DIN0207_L6.3mm_D2.5mm_P7.62mm_Horizontal
- moved J8 59.3 mm to (78.8, 118.9), turned to 0 degrees
- moved TP9 56.5 mm to (31.9, 78.3), turned to 90 degrees
- moved TP10 56.4 mm to (31.9, 97.3), turned to 90 degrees
- moved SW1 51.9 mm to (85.2, 118.8), turned to 90 degrees
- moved U18 43.8 mm to (78.2, 62.8), turned to 0 degrees
- moved R2a1 41.8 mm to (78.2, 59.6)
- moved R1a1 40.9 mm to (74.1, 59.6), turned to 0 degrees
- moved R4a1 38.5 mm to (82.3, 62.8)
- moved U16 38.4 mm to (73.8, 62.8), turned to 180 degrees
- moved U17 36.7 mm to (63.0, 119.5), turned to 0 degrees
- moved SW2 34.3 mm to (207.5, 102.5)
- moved R3a1 33.8 mm to (82.4, 59.6)
- moved R4b1 32.1 mm to (71.6, 118.9)
- moved R3 31.5 mm to (195.8, 84.7), turned to 0 degrees
- moved R26 31.1 mm to (204.5, 91.0), turned to 90 degrees
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Connections:
- N1 pad 1: /Power Distribution/5V_I_SENSE_OP -> 5V_BUS
- N2 pad 1: /Power Distribution/12V_I_SENSE_OP -> 12V_BUS
- Q2 pad 2: GND -> Net-(JP2-Pad2)
- Q2 pad 3: Net-(JP2-Pad2) -> GND
- Q3 pad 2: GND -> Net-(JP3-Pad2)
- Q3 pad 3: Net-(JP3-Pad2) -> GND
- U6 pad 3: /Power Distribution/5V_I_SENSE_OP -> 5V_BUS
- U6 pad 4: /Power Distribution/5V_I_SENSE_OP -> 5V_BUS
- U7 pad 3: /Power Distribution/12V_I_SENSE_OP -> 12V_BUS
- U7 pad 4: /Power Distribution/12V_I_SENSE_OP -> 12V_BUS
Routing:
- net 12V_BUS: track 0.00 -> 341.5 mm
- net 24V_BUS: track 0.00 -> 170.2 mm
- net 5V_BUS: track 0.00 -> 164.2 mm
- net MCU_5V: track 0.00 -> 138.8 mm, vias 0 -> 4
- net /BUS_I_SENSE_A: track 0.00 -> 104.5 mm, vias 0 -> 2
- net /5V_BUS_MONITOR: track 0.00 -> 83.6 mm, vias 0 -> 3
- net Net-(J8-Pad3): track 0.00 -> 48.2 mm, vias 0 -> 1
- net /AtMega328p/MCU_5V_BUS: track 0.00 -> 43.8 mm
- net Net-(J8-Pad4): track 0.00 -> 42.8 mm, vias 0 -> 1
- net /AtMega328p/USB MCU CH340 Interface A/DTR_A: track 0.00 -> 34.6 mm
- net /Power Distribution/5V_I_SENSE_IP: track 0.00 -> 29.8 mm
- net /Power Distribution/12V_I_SENSE_IP: track 0.00 -> 25.2 mm
- net Net-(C25-Pad2): track 0.00 -> 20.4 mm
- net /AtMega328p/CH_G: track 0.00 -> 19.7 mm, vias 0 -> 2
- net /24V_1: track 0.00 -> 15.7 mm
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Other:
- board size 241.8 x 99.1 mm -> 207.4 x 99.1 mm
