File: ISOpowerPCB/ISOpower.kicad_pcb (KiCad board)
At the start: 4 copper layers, 207.4 x 99.1 mm, 189 parts, among them J1 XT60_connector_DC_60A_male, J10 USB_CH_A, J11 USB_CH_A, J12 USB_CH_A, J13 USB_CH_A, J14 XT30_connector_DC_30A_female, J15 XT30_connector_DC_30A_female, J16 XT30_connector_DC_30A_female, J17 XT30_connector_DC_30A_female, J18 XT30_connector_DC_30A_female, J19 ESP32_header, J2 ESP_GPIO_B, J20 USB_B_Mini, J21 24vTerminal, J22 12vTerminal, J23 5vTerminal, J24 dio_spare, J25 adc_spare, J26 USB_5v, J29 wifi_header, J3 ESPpin4-7, J30 3V3_spare, J31 USB_B_Mini, J4 SDI-SDO, J5 ESP_GPIO_A, J6 prog_power_select, J7 i2c Header, J8 AVR-ISP-6, J9 USB_CH_A, M1 Fan_IEC60617, Q1 IRF5305_PBF, Q10 BC817, Q11 BC817, Q12 BC817, Q13 BC817, Q14 BC817, Q15 BC817, Q16 BC817, Q17 BC817, Q18 BC817, Q19 BC817, Q2 Si2319CDS, Q20 BC817, Q3 Si2319CDS, Q4 IRF5305_PBF, Q5 IRF5305_PBF, Q6 IRF5305_PBF, Q7 IRF5305_PBF, Q8 IRF5305_PBF, Q9 BC817, SW1 SW_Push, SW2 BOOT, SW3 EN, U1 ESP32-WROOM-32, U10 LM2596S-5, U13 TXS0102DCT, U14 CH340C, U15 TL431DBZ, U16 TL431DBZ, U17 TL431DBZ, U18 TL431DBZ, U19 HEF4093B, U2 AMS1117-3.3, U3 ATmega328PB-M, U4 i6A4W020A-DC-DC-250W, U5 i6A4W020A-DC-DC-250W, U6 ACS712xLCTR-30A, U7 ACS712xLCTR-30A, U8 CH340C, Y1 16MHz

Commit message: PCB layout completed.
Screenshots added to media folder
Parts:
- added G***: LOGO, 000_Graphics_Immo:UoE_logo5x5, F.Cu at (169.5, 106.0)
- added G***: LOGO, 000_Graphics_Immo:UoE_logo5x5, F.Cu at (258.5, 126.5)
- added G***: LOGO, 000_Graphics_Immo:UoE_logo, B.Cu at (145.4, 89.5)
- added G***: LOGO, 000_Graphics_Immo:UoE_logo25x25, B.Cu at (223.0, 115.0)
- added N3: Net_Tie, NetTie:NetTie-2_SMD_Pad0.5mm, F.Cu at (125.7, 67.5)
- added N4: Net_Tie, NetTie:NetTie-2_SMD_Pad0.5mm, F.Cu at (142.9, 120.7)
- J24: value dio_spare -> PD4
- J25: value adc_spare -> ADC
- J8: value AVR-ISP-6 -> AVR-ISP
- JP2, JP3, JP4, JP5, JP6, JP7, JP8: footprint Jumper:SolderJumper-2_P1.3mm_Open_RoundedPad1.0x1.5mm -> Jumper:SolderJumpermodded1.0x1.5mm
- TP10: value 5V_MONITOR -> 5V_TEST
- TP7: value CH340_UD- -> +UD
- TP8: value CH340_UD+ -> -UD
- moved TP10 64.6 mm to (86.1, 132.4), turned to 180 degrees
- moved TP9 64.2 mm to (95.6, 70.2), turned to 0 degrees
- moved TP6 44.5 mm to (107.0, 133.7), turned to 0 degrees
- moved TP3 34.2 mm to (130.0, 133.2)
- moved R4 33.4 mm to (154.9, 126.7), turned to 0 degrees
- moved U8 32.3 mm to (161.6, 122.3)
- moved C24 30.4 mm to (154.9, 121.6), turned to 180 degrees
- moved C28 30.1 mm to (223.6, 112.5)
- moved C29 30.1 mm to (218.3, 112.5)
- moved C5 30.1 mm to (222.3, 107.6)
- moved D9 30.1 mm to (238.8, 116.5)
- moved H10 30.1 mm to (252.8, 127.1)
- moved H5 30.1 mm to (252.8, 100.4)
- moved J20 30.1 mm to (214.6, 120.1)
- moved Q20 30.1 mm to (232.5, 108.9)
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Connections:
- R12 pad 2: 12V_BUS -> HV
- R13 pad 2: 12V_BUS -> HV
- R14 pad 2: 12V_BUS -> HV
- R18 pad 2: 12V_BUS -> HV
- R19 pad 2: 12V_BUS -> HV
- R20 pad 2: 12V_BUS -> HV
- R23 pad 2: 12V_BUS -> HV
- R35 pad 2: 12V_BUS -> HV
- R38 pad 2: 12V_BUS -> HV
- R39 pad 2: 12V_BUS -> HV
- U3 pad 21: GND -> /AtMega328p/at_gnd
- U3 pad 33: GND -> /AtMega328p/at_gnd
- U3 pad 5: GND -> /AtMega328p/at_gnd
Routing:
- net GND: track 0.00 -> 236.4 mm, vias 0 -> 31
- net /ESP32_Daughterboard/3V3_BUS: track 0.00 -> 119.6 mm, vias 0 -> 3
- net /12V_BUS_MONITOR: track 10.8 -> 129.8 mm, vias 0 -> 3
- net HV: track 0.00 -> 112.3 mm, vias 0 -> 2
- net /Power Outputs/5v to 12v logic conversion_v2/0_OUT: track 0.00 -> 88.4 mm, vias 0 -> 2
- net /ESP32_Daughterboard/GND: track 0.00 -> 84.6 mm, vias 0 -> 13
- net Net-(D8-Pad2): track 0.00 -> 84.5 mm, vias 0 -> 2
- net Net-(D6-Pad2): track 0.00 -> 83.5 mm, vias 0 -> 2
- net /USB_PBUS: track 3.12 -> 76.2 mm, vias 0 -> 2
- net /Power Outputs/5v to 12v logic conversion_v2/1_OUT: track 3.94 -> 73.3 mm, vias 0 -> 2
- net /ESP32_Daughterboard/MCU_5V_BUS: track 0.00 -> 66.1 mm, vias 0 -> 3
- net /BUS_B_DISABLE: track 0.00 -> 62.8 mm, vias 0 -> 2
- net 5V_BUS: track 164.2 -> 225.9 mm
- net /BUS_A_DISABLE: track 0.00 -> 57.3 mm, vias 0 -> 2
- net /Power Outputs/5v to 12v logic conversion_v2/2_OUT: track 3.94 -> 60.6 mm, vias 0 -> 2
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- added copper zone on B.Cu, net /ESP32_Daughterboard/GND
- added copper zone on B.Cu, net GND
Other:
- board size 207.4 x 99.1 mm -> 203.9 x 99.1 mm
- board text added: "+12v"
- board text added: "+24v"
- board text added: "+5v"
- board text added: "4 | 5"
- board text added: "GND"
- board text added: "ISOpower.V1.0."
- board text added: "ISOpower_wifiModule"
- board text added: "V1.0"
- board text added: "out_A"
- board text added: "out_B"
- board text added: "out_C"
- board text added: "out_D"
- board text added: "out_E"
