File: ISOpowerPCB/ISOpower.kicad_pcb (KiCad board)
At the start: 4 copper layers, 119.4 x 99.1 mm, 159 parts, among them J1 XT60_connector_DC_60A_male, J10 USB_CH_A, J11 USB_CH_A, J12 USB_CH_A, J13 USB_CH_A, J14 XT30_connector_DC_30A_female, J15 XT30_connector_DC_30A_female, J16 XT30_connector_DC_30A_female, J17 XT30_connector_DC_30A_female, J18 XT30_connector_DC_30A_female, J21 24vTerminal, J22 12vTerminal, J23 5vTerminal, J24 dio_spare, J25 adc_spare, J26 USB_5v, J29 wifi_header, J30 3V3_spare, J31 USB_B_Mini, J6 prog_power_select, J8 AVR-ISP-6, J9 USB_CH_A, M1 Fan_IEC60617, Q1 IRF5305_PBF, Q10 BC817, Q11 BC817, Q12 BC817, Q13 BC817, Q14 BC817, Q15 BC817, Q16 BC817, Q17 BC817, Q18 BC817, Q2 Si2319CDS, Q3 Si2319CDS, Q4 IRF5305_PBF, Q5 IRF5305_PBF, Q6 IRF5305_PBF, Q7 IRF5305_PBF, Q8 IRF5305_PBF, Q9 BC817, SW1 SW_Push, U10 LM2596S-5, U15 TL431DBZ, U16 TL431DBZ, U17 TL431DBZ, U18 TL431DBZ, U19 HEF4093B, U3 ATmega328PB-M, U4 i6A4W020A-DC-DC-250W, U5 i6A4W020A-DC-DC-250W, U6 ACS712xLCTR-30A, U7 ACS712xLCTR-30A, U8 CH340C, Y1 16MHz

Commit message: Adding fabrication files
Parts:
- J8: footprint Connector_PinHeader_1.27mm:PinHeader_2x03_P1.27mm_Vertical -> Connector_PinHeader_2.54mm:PinHeader_2x03_P2.54mm_Vertical
- moved R3b1 5.76 mm to (92.7, 118.7)
- moved N8 3.42 mm to (98.7, 120.7)
- moved J8 2.22 mm to (104.8, 128.3), turned to 90 degrees
Routing:
- net 5V_BUS: track 277.2 -> 290.1 mm, vias 36 -> 38
- net Net-(R3b1-Pad2): track 17.1 -> 23.8 mm, vias 2 -> 3
- net Net-(N8-Pad2): track 15.3 -> 11.0 mm
- net /AtMega328p/MCU_5V_BUS: track 96.0 -> 99.5 mm
- net Net-(J8-Pad1): track 49.6 -> 52.1 mm, vias 1 -> 2
- net Net-(J8-Pad4): track 45.7 -> 47.2 mm
- net /Power Distribution/5V_I_SENSE_IP: track 42.7 -> 41.6 mm
- net /AtMega328p/USB MCU CH340 Interface A/DTR_A: track 75.8 -> 75.1 mm

Commit message: blegh
Changed lines of the file:
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@@
   (segment (start 164.465 97.79) (end 164.465 95.69952) (width 3.5) (layer "B.Cu") (net 1))
   (segment (start 121.099511 124.409511) (end 121.094511 124.414511) (width 0.3) (layer "F.Cu") (net 2))
-  (segment (start 118.745 103.505) (end 90.229244 103.505) (width 0.3) (layer "F.Cu") (net 2))
   (segment (start 124.46 112.395) (end 122.49 112.395) (width 0.3) (layer "F.Cu") (net 2))
-  (segment (start 89.247122 102.522878) (end 89.247122 107.304687) (width 0.3) (layer "F.Cu") (net 2))
   (segment (start 125.095 107.315) (end 125.73 107.95) (width 0.3) (layer "F.Cu") (net 2))
   (segment (start 125.73 111.125) (end 124.46 112.395) (width 0.3) (layer "F.Cu") (net 2))
@@
   (segment (start 80.088794 114.329511) (end 78.619511 115.798794) (width 0.2) (layer "F.Cu") (net 2))
   (segment (start 78.619511 116.139511) (end 78.619511 115.728084) (width 0.3) (layer "F.Cu") (net 2))
-  (segment (start 86.344511 110.207298) (end 86.344511 112.899511) (width 0.3) (layer "F.Cu") (net 2))
+  (segment (start 90.043 106.508809) (end 90.043 103.251) (width 0.3) (layer "F.Cu") (net 2))
   (segment (start 121.094511 124.414511) (end 117.924511 124.414511) (width 0.3) (layer "F.Cu") (net 2))
   (segment (start 75.924283 75.565) (end 73.782914 73.423631) (width 0.2) (layer "F.Cu") (net 2))
@@
   (segment (start 130.81 111.76) (end 131.41597 112.36597) (width 0.3) (layer "F.Cu") (net 2))
   (segment (start 127.635 122.555) (end 122.954022 122.555) (width 0.3) (layer "F.Cu") (net 2))
+  (segment (start 86.344511 110.207298) (end 90.043 106.508809) (width 0.3) (layer "F.Cu") (net 2))
   (segment (start 84.944022 114.3) (end 83.231029 114.3) (width 0.3) (layer "F.Cu") (net 2))
   (segment (start 155.29452 89.371671) (end 154.943329 89.02048) (width 0.3) (layer "F.Cu") (net 2))
   (segment (start 155.29452 89.88952) (end 155.29452 89.371671) (width 0.3) (layer "F.Cu") (net 2))
-  (segment (start 89.247122 107.304687) (end 86.344511 110.207298) (width 0.3) (layer "F.Cu") (net 2))
   (segment (start 131.740489 118.449511) (end 127.635 122.555) (width 0.3) (layer "F.Cu") (net 2))
-  (segment (start 90.229244 103.505) (end 89.247122 102.522878) (width 0.3) (layer "F.Cu") (net 2))
   (segment (start 83.231029 114.3) (end 83.116528 114.185499) (width 0.3) (layer "F.Cu") (net 2))
   (segment (start 154.943329 89.02048) (end 148.94452 89.02048) (width 0.3) (layer "F.Cu") (net 2))
   (segment (start 86.344511 112.899511) (end 85.045 114.199022) (width 0.2) (layer "F.Cu") (net 2))
+  (segment (start 125.095 97.155) (end 118.745 103.505) (width 0.3) (layer "F.Cu") (net 2))
   (segment (start 133.054511 114.639511) (end 133.023088 114.670934) (width 0.3) (layer "F.Cu") (net 2))
   (segment (start 145.385 92.58) (end 133.48 92.58) (width 0.3) (layer "F.Cu") (net 2))
@@
   (segment (start 122.954022 122.555) (end 121.099511 124.409511) (width 0.3) (layer "F.Cu") (net 2))
   (segment (start 122.49 112.395) (end 121.855 113.03) (width 0.3) (layer "F.Cu") (net 2))
+  (segment (start 118.745 103.505) (end 90.297 103.505) (width 0.3) (layer "F.Cu") (net 2))
   (segment (start 80.047595 114.3) (end 81.915 114.3) (width 0.3) (layer "F.Cu") (net 2))
   (segment (start 81.818275 114.329511) (end 81.309511 114.329511) (width 0.2) (layer "F.Cu") (net 2))
   (segment (start 83.116528 114.185499) (end 82.495618 114.185499) (width 0.3) (layer "F.Cu") (net 2))
-  (segment (start 125.095 97.155) (end 118.745 103.505) (width 0.3) (layer "F.Cu") (net 2))
   (segment (start 127 112.395) (end 127.635 112.395) (width 0.3) (layer "F.Cu") (net 2))
+  (segment (start 90.297 103.505) (end 90.043 103.251) (width 0.3) (layer "F.Cu") (net 2))
   (segment (start 125.095 97.155) (end 125.095 107.315) (width 0.3) (layer "F.Cu") (net 2))
   (segment (start 133.48 92.58) (end 129.67 92.58) (width 0.3) (layer "F.Cu") (net 2))
   (segment (start 147.795 90.17) (end 145.385 92.58) (width 0.3) (layer "F.Cu") (net 2))
   (segment (start 129.67 92.58) (end 125.095 97.155) (width 0.3) (layer "F.Cu") (net 2))
+  (segment (start 86.344511 112.899511) (end 86.344511 110.207298) (width 0.3) (layer "F.Cu") (net 2))
   (segment (start 86.344511 112.899511) (end 84.944022 114.3) (width 0.3) (layer "F.Cu") (net 2))
   (segment (start 129.54 111.76) (end 130.81 111.76) (width 0.3) (layer "F.Cu") (net 2))
@@
   (segment (start 129.319511 111.980489) (end 129.54 111.76) (width 0.3) (layer "F.Cu") (net 2))
   (via (at 73.66 76.835) (size 0.8) (drill 0.4) (layers "F.Cu" "B.Cu") (net 2))
-  (via (at 89.247122 102.522878) (size 0.8) (drill 0.4) (layers "F.Cu" "B.Cu") (net 2))
-  (segment (start 73.66 86.935756) (end 73.66 76.835) (width 0.3) (layer "In2.Cu") (net 2))
-  (segment (start 89.247122 102.522878) (end 73.66 86.935756) (width 0.3) (layer "In2.Cu") (net 2))
+  (via (at 90.043 103.251) (size 0.8) (drill 0.4) (layers "F.Cu" "B.Cu") (net 2))
+  (segment (start 73.66 86.935756) (end 89.975244 103.251) (width 0.3) (layer "In2.Cu") (net 2))
+  (segment (start 89.975244 103.251) (end 90.043 103.251) (width 0.3) (layer "In2.Cu") (net 2))
+  (segment (start 73.66 76.835) (end 73.66 86.935756) (width 0.3) (layer "In2.Cu") (net 2))
   (segment (start 140.418533 120.354511) (end 138.769511 120.354511) (width 0.2) (layer "F.Cu") (net 3))
   (segment (start 138.134511 114.639511) (end 138.134511 118.619511) (width 0.2) (layer "F.Cu") (net 3))
@@
   (segment (start 122.084511 119.215489) (end 122.413043 119.544021) (width 0.2) (layer "In2.Cu") (net 49))
   (segment (start 144.129825 117.522288) (end 144.080499 117.571614) (width 0.2) (layer "F.Cu") (net 50))
+  (segment (start 132.947862 112.97) (end 143.45 112.97) (width 0.2) (layer "F.Cu") (net 50))
   (segment (start 131.445 108.585) (end 132.264991 109.404991) (width 0.2) (layer "F.Cu") (net 50))
   (segment (start 144.080499 117.571614) (end 144.080499 118.151102) (width 0.2) (layer "F.Cu") (net 50))
@@
   (segment (start 144.533908 118.604511) (end 145.222011 118.604511) (width 0.2) (layer "F.Cu") (net 50))
   (segment (start 143.45 112.97) (end 144.129825 113.649825) (width 0.2) (layer "F.Cu") (net 50))
-  (segment (start 132.947862 112.97) (end 143.45 112.97) (width 0.2) (layer "F.Cu") (net 50))
   (segment (start 132.264991 112.287128) (end 132.947862 112.97) (width 0.2) (layer "F.Cu") (net 50))
   (segment (start 144.129825 113.649825) (end 144.129825 117.522288) (width 0.2) (layer "F.Cu") (net 50))
@@
   (segment (start 155.445998 126.365) (end 161.29 126.365) (width 0.3) (layer "In1.Cu") (net 99))
   (segment (start 129.205 128.597294) (end 132.965 128.597294) (width 0.3) (layer "In1.Cu") (net 99))
-  (segment (start 139.529022 115.665) (end 139.16 115.665) (width 0.2) (layer "F.Cu") (net 100))
-  (segment (start 131.63153 111.945826) (end 131.63153 110.742035) (width 0.2) (layer "F.Cu") (net 100))
-  (segment (start 145.222011 119.104511) (end 142.968533 119.104511) (width 0.2) (layer "F.Cu") (net 100))
-  (segment (start 142.968533 119.104511) (end 139.529022 115.665) (width 0.2) (layer "F.Cu") (net 100))
-  (segment (start 139.16 115.665) (end 139.16 113.879808) (width 0.2) (layer "F.Cu") (net 100))
-  (segment (start 138.650192 113.37) (end 132.782869 113.37) (width 0.2) (layer "F.Cu") (net 100))
-  (segment (start 131.86548 112.179776) (end 131.63153 111.945826) (width 0.2) (layer "F.Cu") (net 100))
-  (segment (start 131.63153 110.742035) (end 128.905 108.015505) (width 0.2) (layer "F.Cu") (net 100))
-  (segment (start 139.16 113.879808) (end 138.650192 113.37) (width 0.2) (layer "F.Cu") (net 100))
-  (segment (start 128.905 108.015505) (end 128.905 106.68) (width 0.2) (layer "F.Cu") (net 100))
-  (segment (start 131.86548 112.452611) (end 131.86548 112.179776) (width 0.2) (layer "F.Cu") (net 100))
-  (segment (start 132.782869 113.37) (end 131.86548 112.452611) (width 0.2) (layer "F.Cu") (net 100))
+  (segment (start 139.16 113.879808) (end 139.16 115.295978) (width 0.2) (layer "F.Cu") (net 100))
+  (segment (start 131.63153 111.945826) (end 131.86548 112.179776) (width 0.2) (layer "F.Cu") (net 100))
+  (segment (start 131.86548 112.179776) (end 131.86548 112.452611) (width 0.2) (layer "F.Cu") (net 100))
+  (segment (start 128.905 108.015505) (end 131.63153 110.742035) (width 0.2) (layer "F.Cu") (net 100))
+  (segment (start 128.905 106.68) (end 128.905 108.015505) (width 0.2) (layer "F.Cu") (net 100))
+  (segment (start 138.650192 113.37) (end 139.16 113.879808) (width 0.2) (layer "F.Cu") (net 100))
+  (segment (start 131.86548 112.452611) (end 132.782869 113.37) (width 0.2) (layer "F.Cu") (net 100))
+  (segment (start 142.968533 119.104511) (end 145.222011 119.104511) (width 0.2) (layer "F.Cu") (net 100))
+  (segment (start 131.63153 110.742035) (end 131.63153 111.945826) (width 0.2) (layer "F.Cu") (net 100))
+  (segment (start 132.782869 113.37) (end 138.650192 113.37) (width 0.2) (layer "F.Cu") (net 100))
+  (segment (start 139.16 115.295978) (end 142.968533 119.104511) (width 0.2) (layer "F.Cu") (net 100))
   (segment (start 147.909511 117.917011) (end 147.909511 116.999517) (width 0.2) (layer "F.Cu") (net 101))
   (segment (start 147.930008 116.97902) (end 147.930008 115.909511) (width 0.2) (layer "F.Cu") (net 101))
