File: ISOpowerPCB/ISOpower_Outputs.kicad_sch (KiCad schematic)
At the start: 23 parts, among them J10 USB_CH_A, J11 USB_CH_A, J12 USB_CH_A, J13 USB_CH_A, J14 XT30_connector_DC_30A_female, J15 XT30_connector_DC_30A_female, J16 XT30_connector_DC_30A_female, J17 XT30_connector_DC_30A_female, J18 XT30_connector_DC_30A_female, J9 USB_CH_A, Q4 IRF5305_PBF, Q5 IRF5305_PBF, Q6 IRF5305_PBF, Q7 IRF5305_PBF, Q8 IRF5305_PBF

Commit message: almost finished needs to pass DRC check and fix aesthetics
Parts:
- N11: footprint NetTie:NetTie-8-15A_1oz_2oz -> NetTie:NetTie-8-15A_1oz_2oz_chamf
Connections:
- net GND: no longer J10.4 (GND), J10.5 (Shield), J11.4 (GND), J11.5 (Shield), J12.4 (GND), J12.5 (Shield), J13.4 (GND), J13.5 (Shield), J14.1 (V-), J15.1 (V-), J16.1 (V-), J17.1 (V-), J18.1 (V-), J9.4 (GND), J9.5 (Shield)
- new net PWR_GND: J10.4 (GND), J10.5 (Shield), J11.4 (GND), J11.5 (Shield), J12.4 (GND), J12.5 (Shield), J13.4 (GND), J13.5 (Shield), J14.1 (V-), J15.1 (V-), J16.1 (V-), J17.1 (V-), J18.1 (V-), J9.4 (GND), J9.5 (Shield)
Other:
- sheet 5v to 12v logic conversion_v2 ports: added PWR_GND; removed none
