File: ISOpowerPCB/ISOpower_distribution.kicad_sch (KiCad schematic)
At the start: 29 parts, among them M1 Fan_IEC60617, Q2 Si2319CDS, Q3 Si2319CDS, U10 LM2596S-5, U4 i6A4W020A-DC-DC-250W, U5 i6A4W020A-DC-DC-250W, U6 ACS712xLCTR-30A, U7 ACS712xLCTR-30A

Commit message: almost finished needs to pass DRC check and fix aesthetics
Parts:
- removed N2: Net_Tie, NetTie:NetTie-2_SMD_Pad0.5mm, symbol 000_Utility_Immo:Net_Tie
Connections:
- net +5V: no longer C15.1, C16.1, U6.8 (VCC), U7.8 (VCC)
- net GND: no longer C10.2, C11.2, C12.2, C13.2, C14.2, C16.2, C17.2, C18.2, C19.2, C20.2, C21.2, C9.2, D3.2 (A), JP2.1 (A), JP3.1 (A), M1.2 (-), Q2.3 (D), Q3.3 (D), R6.2, R7.2, U10.3 (GND), U10.5 (~{ON}/OFF), U4.3 (Vin(-)), U4.4 (Vout(-)), U5.3 (Vin(-)), U5.4 (Vout(-)), U6.5 (GND), U7.5 (GND)
- net MCU_5V_OUT: now also C15.1, C16.1, U6.8 (VCC), U7.8 (VCC)
- new net GND_PWR: C10.2, C11.2, C12.2, C13.2, C14.2, C16.2, C17.2, C18.2, C19.2, C20.2, C21.2, C9.2, D3.2 (A), JP2.1 (A), JP3.1 (A), M1.2 (-), Q2.3 (D), Q3.3 (D), R6.2, R7.2, U10.3 (GND), U10.5 (~{ON}/OFF), U4.3 (Vin(-)), U4.4 (Vout(-)), U5.3 (Vin(-)), U5.4 (Vout(-)), U6.5 (GND), U7.5 (GND)
