File: ISOpowerPCB/ISOpower_distribution.kicad_sch (KiCad schematic)
At the start: 28 parts, among them M1 Fan_IEC60617, Q2 Si2319CDS, Q3 Si2319CDS, U10 LM2596S-5, U4 i6A4W020A-DC-DC-250W, U5 i6A4W020A-DC-DC-250W, U6 ACS712xLCTR-30A, U7 ACS712xLCTR-30A

Commit message: blegh
Connections:
- net +24V: no longer U5.1 (Vin(+))
- net 12V_I_SENSE_IP: no longer U5.7 (Sense(+)), U5.8 (Vout(+))
- net GND_PWR: no longer U5.3 (Vin(-)), U5.4 (Vout(-))
- net at R7.1: no longer U5.6 (Trim)
- net at JP3.2 (B), Q3.2 (S): no longer U5.2 (On/Off)
Other:
- moved on the sheet: U5
Changed lines of the file:
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@@
     (pin "3")
   )
-  (symbol (lib_id "000_Modules_Immo:i6A4W020A-DC-DC-250W") (at 80.01 67.31 0) (unit 1)
+  (symbol (lib_id "000_Modules_Immo:i6A4W020A-DC-DC-250W") (at 80.01 67.31 0) (mirror y) (unit 1)
     (in_bom yes) (on_board yes) (fields_autoplaced)
-    (property "Reference" "U5" (id 0) (at 79.375 57.15 0))
-    (property "Value" "i6A4W020A-DC-DC-250W" (id 1) (at 79.375 59.69 0))
+    (property "Reference" "U5" (id 0) (at 80.645 57.15 0))
+    (property "Value" "i6A4W020A-DC-DC-250W" (id 1) (at 80.645 59.69 0))
     (property "Footprint" "ISOpower:i6A4W-DIP" (id 2) (at 80.01 67.31 0)
       (effects (font (size 1.27 1.27)) hide)
