File: ISOpowerPCB/ISOpower-backups/ISOpower-2022-03-02_161759/ISOpower.kicad_pcb (KiCad board)
At the start: 4 copper layers, 199.9 x 99.1 mm, 192 parts, among them J1 XT60_connector_DC_60A_male, J10 USB_CH_A, J11 USB_CH_A, J12 USB_CH_A, J13 USB_CH_A, J14 XT30_connector_DC_30A_female, J15 XT30_connector_DC_30A_female, J16 XT30_connector_DC_30A_female, J17 XT30_connector_DC_30A_female, J18 XT30_connector_DC_30A_female, J19 ESP32_header, J2 ESP_GPIO_B, J20 USB_B_Mini, J21 24vTerminal, J22 12vTerminal, J23 5vTerminal, J24 dio_spare, J25 adc_spare, J26 USB_5v, J29 wifi_header, J3 ESPpin4-7, J30 3V3_spare, J31 USB_B_Mini, J4 SDI-SDO, J5 ESP_GPIO_A, J6 prog_power_select, J7 i2c Header, J8 AVR-ISP-6, J9 USB_CH_A, M1 Fan_IEC60617, Q1 IRF5305_PBF, Q10 BC817, Q11 BC817, Q12 BC817, Q13 BC817, Q14 BC817, Q15 BC817, Q16 BC817, Q17 BC817, Q18 BC817, Q19 BC817, Q2 Si2319CDS, Q20 BC817, Q3 Si2319CDS, Q4 IRF5305_PBF, Q5 IRF5305_PBF, Q6 IRF5305_PBF, Q7 IRF5305_PBF, Q8 IRF5305_PBF, Q9 BC817, SW1 SW_Push, SW2 BOOT, SW3 EN, U1 ESP32-WROOM-32, U10 LM2596S-5, U13 TXS0102DCT, U14 CH340C, U15 TL431DBZ, U16 TL431DBZ, U17 TL431DBZ, U18 TL431DBZ, U19 HEF4093B, U2 AMS1117-3.3, U3 ATmega328PB-M, U4 i6A4W020A-DC-DC-250W, U5 i6A4W020A-DC-DC-250W, U6 ACS712xLCTR-30A, U7 ACS712xLCTR-30A, U8 CH340C, Y1 16MHz

Commit message: almost finished needs to pass DRC check and fix aesthetics
Changed lines of the file:
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@@
     (fp_line (start -3.95 -2) (end 3.95 -2) (layer "F.CrtYd") (width 0.05))
     (fp_line (start -3.95 2) (end -3.95 -2) (layer "F.CrtYd") (width 0.05))
+    (fp_line (start 3 1.75) (end -3 1.75) (layer "F.Fab") (width 0.1))
     (fp_line (start -3 -1.75) (end 3 -1.75) (layer "F.Fab") (width 0.1))
+    (fp_line (start 3 -1.75) (end 3 1.75) (layer "F.Fab") (width 0.1))
     (fp_line (start 1.4 -0.7) (end 1.4 0.7) (layer "F.Fab") (width 0.1))
     (fp_line (start -3 1.75) (end -3 -1.75) (layer "F.Fab") (width 0.1))
@@
     (fp_line (start -1.4 -0.7) (end 1.4 -0.7) (layer "F.Fab") (width 0.1))
     (fp_line (start 1.4 0.7) (end -1.4 0.7) (layer "F.Fab") (width 0.1))
-    (fp_line (start 3 1.75) (end -3 1.75) (layer "F.Fab") (width 0.1))
-    (fp_line (start 3 -1.75) (end 3 1.75) (layer "F.Fab") (width 0.1))
     (pad "1" smd rect locked (at -2.7 0 180) (size 2 1.6) (layers "F.Cu" "F.Paste" "F.Mask")
       (net 1 "/ESP32_Daughterboard/USB ESP32 CH340 Interface /ESP_EN") (pinfunction "1") (pintype "passive"))
@@
   (gr_line (start 177.506159 94.527841) (end 129.54 94.488) (layer "F.SilkS") (width 0.15))
   (gr_line (start 179.451 128.651) (end 179.451 96.52) (layer "F.SilkS") (width 0.15))
-  (gr_arc (start 177.379159 94.527841) (mid 178.858898 95.06235) (end 179.451 96.52) (layer "F.SilkS") (width 0.15))
+  (gr_arc (start 177.379159 94.527841) (mid 178.859167 95.062609) (end 179.451 96.52) (layer "F.SilkS") (width 0.15))
   (gr_arc (start 179.451 128.651) (mid 178.976831 129.663498) (end 177.927 130.048) (layer "F.SilkS") (width 0.15))
   (gr_rect (start 87.31 119.615) (end 99.422781 128.59) (layer "F.SilkS") (width 0.15) (fill none))
